File: boards/spine/spine-fpga.sch (KiCad schematic (older format))
At the start: 24 parts, among them U7 iCE40-HX1K-TQ144

Commit message: Power management and such
Parts:
- renumbered C29 to C30, C30 to C31, C31 to C32, C32 to C33, C33 to C34, C34 to C35, C35 to C36, C36 to C37, C37 to C38, C38 to C39, C39 to C40, C40 to C41, C41 to C42, C42 to C43, C43 to C44, C44 to C45, C45 to C46, C46 to C47
Changed lines of the file:
@@
 $EndComp
 $Comp
-L GND #PWR112
+L GND #PWR0105
 U 1 1 56403C36
 P 3050 1550
-F 0 "#PWR112" H 3050 1300 50  0001 C CNN
+F 0 "#PWR0105" H 3050 1300 50  0001 C CNN
 F 1 "GND" V 3050 1350 50  0000 C CNN
 F 2 "" H 3050 1550 60  0000 C CNN
@@
 $EndComp
 $Comp
-L +1V2 #PWR113
+L +1V2 #PWR0106
 U 1 1 564083AC
 P 3050 1850
-F 0 "#PWR113" H 3050 1700 50  0001 C CNN
+F 0 "#PWR0106" H 3050 1700 50  0001 C CNN
 F 1 "+1V2" V 3050 2050 50  0000 C CNN
 F 2 "" H 3050 1850 60  0000 C CNN
@@
 	2100 1250 2100 1950
 $Comp
-L +1V2 #PWR109
+L +1V2 #PWR0107
 U 1 1 5640879A
 P 2100 950
-F 0 "#PWR109" H 2100 800 50  0001 C CNN
+F 0 "#PWR0107" H 2100 800 50  0001 C CNN
 F 1 "+1V2" H 2100 1100 50  0000 C CNN
 F 2 "" H 2100 950 60  0000 C CNN
@@
 NoConn ~ 3050 2150
 $Comp
-L +3V3 #PWR118
+L +3V3 #PWR0108
 U 1 1 5640CF73
 P 6150 6450
-F 0 "#PWR118" H 6150 6300 50  0001 C CNN
+F 0 "#PWR0108" H 6150 6300 50  0001 C CNN
 F 1 "+3V3" V 6150 6700 50  0000 C CNN
 F 2 "" H 6150 6450 60  0000 C CNN
@@
 SPI_SS
 $Comp
-L +3V3 #PWR110
+L +3V3 #PWR0109
 U 1 1 5640D6CD
 P 2600 2900
-F 0 "#PWR110" H 2600 2750 50  0001 C CNN
+F 0 "#PWR0109" H 2600 2750 50  0001 C CNN
 F 1 "+3V3" H 2600 3040 50  0000 C CNN
 F 2 "" H 2600 2900 60  0000 C CNN
@@
 Connection ~ 2600 3050
 $Comp
-L GND #PWR111
+L GND #PWR0110
 U 1 1 5640DE11
 P 2600 4500
-F 0 "#PWR111" H 2600 4250 50  0001 C CNN
+F 0 "#PWR0110" H 2600 4250 50  0001 C CNN
 F 1 "GND" H 2600 4350 50  0000 C CNN
 F 2 "" H 2600 4500 60  0000 C CNN
@@
 $EndComp
 $Comp
-L +3V3 #PWR117
+L +3V3 #PWR0111
 U 1 1 5640E61C
 P 6150 3200
-F 0 "#PWR117" H 6150 3050 50  0001 C CNN
+F 0 "#PWR0111" H 6150 3050 50  0001 C CNN
 F 1 "+3V3" V 6150 3450 50  0000 C CNN
 F 2 "" H 6150 3200 60  0000 C CNN
@@
 $EndComp
 $Comp
-L +3V3 #PWR120
+L +3V3 #PWR0112
 U 1 1 5640E78F
 P 8750 3400
-F 0 "#PWR120" H 8750 3250 50  0001 C CNN
+F 0 "#PWR0112" H 8750 3250 50  0001 C CNN
 F 1 "+3V3" V 8750 3650 50  0000 C CNN
 F 2 "" H 8750 3400 60  0000 C CNN
@@
 $EndComp
 $Comp
-L +3V3 #PWR121
+L +3V3 #PWR0113
 U 1 1 5640E7E2
 P 8750 6450
-F 0 "#PWR121" H 8750 6300 50  0001 C CNN
+F 0 "#PWR0113" H 8750 6300 50  0001 C CNN
 F 1 "+3V3" V 8750 6700 50  0000 C CNN
 F 2 "" H 8750 6450 60  0000 C CNN
@@
 $EndComp
 $Comp
-L +1V2 #PWR105
+L +1V2 #PWR0114
 U 1 1 5640EE64
 P 1950 5250
-F 0 "#PWR105" H 1950 5100 50  0001 C CNN
+F 0 "#PWR0114" H 1950 5100 50  0001 C CNN
 F 1 "+1V2" H 1950 5400 50  0000 C CNN
 F 2 "" H 1950 5250 60  0000 C CNN
@@
 $EndComp
 $Comp
-L +3V3 #PWR107
+L +3V3 #PWR0115
 U 1 1 5640F3E2
 P 1950 6500
-F 0 "#PWR107" H 1950 6350 50  0001 C CNN
+F 0 "#PWR0115" H 1950 6350 50  0001 C CNN
 F 1 "+3V3" H 1950 6640 50  0000 C CNN
 F 2 "" H 1950 6500 60  0000 C CNN
@@
 Connection ~ 4750 7100
 $Comp
-L GND #PWR106
+L GND #PWR0116
 U 1 1 5640FDCB
 P 1950 5950
-F 0 "#PWR106" H 1950 5700 50  0001 C CNN
+F 0 "#PWR0116" H 1950 5700 50  0001 C CNN
 F 1 "GND" H 1950 5800 50  0000 C CNN
 F 2 "" H 1950 5950 60  0000 C CNN
@@
 $EndComp
 $Comp
-L GND #PWR108
+L GND #PWR0117
 U 1 1 5640FE24
 P 1950 7200
-F 0 "#PWR108" H 1950 6950 50  0001 C CNN
+F 0 "#PWR0117" H 1950 6950 50  0001 C CNN
 F 1 "GND" H 1950 7050 50  0000 C CNN
 F 2 "" H 1950 7200 60  0000 C CNN
@@
 Connection ~ 8450 4350
 $Comp
-L +3V3 #PWR119
+L +3V3 #PWR0118
 U 1 1 56410A99
 P 8250 3750
-F 0 "#PWR119" H 8250 3600 50  0001 C CNN
+F 0 "#PWR0118" H 8250 3600 50  0001 C CNN
 F 1 "+3V3" H 8250 3890 50  0000 C CNN
 F 2 "" H 8250 3750 60  0000 C CNN
@@
 CRESET_B
 $Comp
-L C C30
+L C C31
 U 1 1 5642DE6C
 P 1950 6850
-F 0 "C30" H 1950 6750 50  0000 L CNN
+F 0 "C31" H 1950 6750 50  0000 L CNN
 F 1 "0.1uF" H 1950 6700 50  0000 L TNN
 F 2 "0805" H 1988 6700 30  0001 C CNN
@@
 $EndComp
 $Comp
-L C C34
+L C C35
 U 1 1 5642DE7E
 P 2350 1650
-F 0 "C34" V 2400 1700 50  0000 L CNN
+F 0 "C35" V 2400 1700 50  0000 L CNN
 F 1 "10uF " V 2400 1350 50  0000 L CNN
 F 2 "1206" H 2388 1500 30  0001 C CNN
@@
 $EndComp
 $Comp
-L C C32
+L C C33
 U 1 1 5642EC58
 P 2300 6850
-F 0 "C32" H 2300 6750 50  0000 L CNN
+F 0 "C33" H 2300 6750 50  0000 L CNN
 F 1 "0.1uF" H 2300 6700 50  0000 L TNN
 F 2 "0805" H 2338 6700 30  0001 C CNN
@@
 $EndComp
 $Comp
-L C C36
+L C C37
 U 1 1 5642ECA2
 P 2650 6850
-F 0 "C36" H 2650 6750 50  0000 L CNN
+F 0 "C37" H 2650 6750 50  0000 L CNN
 F 1 "0.1uF" H 2650 6700 50  0000 L TNN
 F 2 "0805" H 2688 6700 30  0001 C CNN
@@
 $EndComp
 $Comp
-L C C38
+L C C39
 U 1 1 5642ECF1
 P 3000 6850
-F 0 "C38" H 3000 6750 50  0000 L CNN
+F 0 "C39" H 3000 6750 50  0000 L CNN
 F 1 "0.1uF" H 3000 6700 50  0000 L TNN
 F 2 "0805" H 3038 6700 30  0001 C CNN
@@
 $EndComp
 $Comp
-L C C40
+L C C41
 U 1 1 5642ED41
 P 3350 6850
-F 0 "C40" H 3350 6750 50  0000 L CNN
+F 0 "C41" H 3350 6750 50  0000 L CNN
 F 1 "0.1uF" H 3350 6700 50  0000 L TNN
 F 2 "0805" H 3388 6700 30  0001 C CNN
@@
 $EndComp
 $Comp
-L C C41
+L C C42
 U 1 1 5642ED94
 P 3700 6850
-F 0 "C41" H 3700 6750 50  0000 L CNN
+F 0 "C42" H 3700 6750 50  0000 L CNN
 F 1 "0.1uF" H 3700 6700 50  0000 L TNN
 F 2 "0805" H 3738 6700 30  0001 C CNN
@@
 $EndComp
 $Comp
-L C C43
+L C C44
 U 1 1 5642EDED
 P 4050 6850
-F 0 "C43" H 4050 6750 50  0000 L CNN
+F 0 "C44" H 4050 6750 50  0000 L CNN
 F 1 "0.1uF" H 4050 6700 50  0000 L TNN
 F 2 "0805" H 4088 6700 30  0001 C CNN
@@
 $EndComp
 $Comp
-L C C44
+L C C45
 U 1 1 5642EE46
 P 4400 6850
-F 0 "C44" H 4400 6750 50  0000 L CNN
+F 0 "C45" H 4400 6750 50  0000 L CNN
 F 1 "0.1uF" H 4400 6700 50  0000 L TNN
 F 2 "0805" H 4438 6700 30  0001 C CNN
@@
 $EndComp
 $Comp
-L C C45
+L C C46
 U 1 1 5642EEA2
 P 4750 6850
-F 0 "C45" H 4750 6750 50  0000 L CNN
+F 0 "C46" H 4750 6750 50  0000 L CNN
 F 1 "0.1uF" H 4750 6700 50  0000 L TNN
 F 2 "0805" H 4788 6700 30  0001 C CNN
@@
 $EndComp
 $Comp
-L C C46
+L C C47
 U 1 1 5642EF02
 P 5100 6850
-F 0 "C46" H 5100 6750 50  0000 L CNN
+F 0 "C47" H 5100 6750 50  0000 L CNN
 F 1 "0.1uF" H 5100 6700 50  0000 L TNN
 F 2 "0805" H 5138 6700 30  0001 C CNN
@@
 $EndComp
 $Comp
-L C C39
+L C C40
 U 1 1 5642EF64
 P 3350 5600
-F 0 "C39" H 3350 5500 50  0000 L CNN
+F 0 "C40" H 3350 5500 50  0000 L CNN
 F 1 "0.1uF" H 3350 5450 50  0000 L TNN
 F 2 "0805" H 3388 5450 30  0001 C CNN
@@
 $EndComp
 $Comp
-L C C37
+L C C38
 U 1 1 5642EFD9
 P 3000 5600
-F 0 "C37" H 3000 5500 50  0000 L CNN
+F 0 "C38" H 3000 5500 50  0000 L CNN
 F 1 "0.1uF" H 3000 5450 50  0000 L TNN
 F 2 "0805" H 3038 5450 30  0001 C CNN
@@
 $EndComp
 $Comp
-L C C35
+L C C36
 U 1 1 5642F044
 P 2650 5600
-F 0 "C35" H 2650 5500 50  0000 L CNN
+F 0 "C36" H 2650 5500 50  0000 L CNN
 F 1 "0.1uF" H 2650 5450 50  0000 L TNN
 F 2 "0805" H 2688 5450 30  0001 C CNN
@@
 $EndComp
 $Comp
-L C C31
+L C C32
 U 1 1 5642F0AF
 P 2300 5600
-F 0 "C31" H 2300 5500 50  0000 L CNN
+F 0 "C32" H 2300 5500 50  0000 L CNN
 F 1 "0.1uF" H 2300 5450 50  0000 L TNN
 F 2 "0805" H 2338 5450 30  0001 C CNN
@@
 $EndComp
 $Comp
-L C C29
+L C C30
 U 1 1 5642F11D
 P 1950 5600
-F 0 "C29" H 1950 5500 50  0000 L CNN
+F 0 "C30" H 1950 5500 50  0000 L CNN
 F 1 "0.1uF" H 1950 5450 50  0000 L TNN
 F 2 "0805" H 1988 5450 30  0001 C CNN
@@
 $EndComp
 $Comp
-L C C33
+L C C34
 U 1 1 5642F812
 P 2350 1400
-F 0 "C33" V 2300 1200 50  0000 L CNN
+F 0 "C34" V 2300 1200 50  0000 L CNN
 F 1 "0.1uF" V 2300 1450 50  0000 L CNN
 F 2 "0805" H 2388 1250 30  0001 C CNN
@@
 Connection ~ 2650 1650
 $Comp
-L +2V5 #PWR114
+L +2V5 #PWR0119
 U 1 1 5644292C
 P 3050 2050
-F 0 "#PWR114" H 3050 1900 50  0001 C CNN
+F 0 "#PWR0119" H 3050 1900 50  0001 C CNN
 F 1 "+2V5" V 3050 2250 50  0000 C CNN
 F 2 "" H 3050 2050 60  0000 C CNN
@@
 	3900 5750 3900 5950
 $Comp
-L GND #PWR116
+L GND #PWR0120
 U 1 1 56443449
 P 3900 5950
-F 0 "#PWR116" H 3900 5700 50  0001 C CNN
+F 0 "#PWR0120" H 3900 5700 50  0001 C CNN
 F 1 "GND" H 3900 5800 50  0000 C CNN
 F 2 "" H 3900 5950 60  0000 C CNN
@@
 $EndComp
 $Comp
-L C C42
+L C C43
 U 1 1 56443455
 P 3900 5600
-F 0 "C42" H 3900 5500 50  0000 L CNN
+F 0 "C43" H 3900 5500 50  0000 L CNN
 F 1 "0.1uF" H 3900 5450 50  0000 L TNN
 F 2 "0805" H 3938 5450 30  0001 C CNN
@@
 $EndComp
 $Comp
-L +2V5 #PWR115
+L +2V5 #PWR0121
 U 1 1 56443529
 P 3900 5250
-F 0 "#PWR115" H 3900 5100 50  0001 C CNN
+F 0 "#PWR0121" H 3900 5100 50  0001 C CNN
 F 1 "+2V5" H 3900 5390 50  0000 C CNN
 F 2 "" H 3900 5250 60  0000 C CNN
@@
 	1    0    0    -1
 $EndComp
+Text HLabel 4700 2550 0    60   BiDi ~ 0
+FIFO_DATA[0..7]
+Text HLabel 4700 2700 0    60   Input ~ 0
+FIFO_RXF#
+Text HLabel 4700 2800 0    60   Input ~ 0
+FIFO_TXE#
+Text HLabel 4700 2900 0    60   Output ~ 0
+FIFO_RD#
+Text HLabel 4700 3000 0    60   Output ~ 0
+FIFO_WR#
+Text HLabel 4700 3150 0    60   Output ~ 0
+FIFO_SIWU
+Text HLabel 4700 3300 0    60   Input ~ 0
+FIFO_CLKOUT
+Text HLabel 4700 3450 0    60   Output ~ 0
+FIFO_OE#
+Text HLabel 4700 3650 0    60   Output ~ 0
+DMX_GATE1
+Text HLabel 4700 3750 0    60   Output ~ 0
+DMX_GATE2
+Text HLabel 4700 3950 0    60   Output ~ 0
+DMX_TX1
+Text HLabel 4700 4050 0    60   Output ~ 0
+DMX_TX2
+Text HLabel 4800 4700 0    60   Output ~ 0
+VBUS_DOWNSTREAM_EN
 $EndSCHEMATC
