File: boards/spine/spine-modules.sch (KiCad schematic (older format))
At the start: 7 parts

Commit message: Getting the FPGA set up
Parts:
- renumbered MOD5 to MOD2, MOD2 to MOD3, MOD6 to MOD4, MOD3 to MOD5, MOD7 to MOD6, MOD4 to MOD7

Commit message: Clock generator, sync connectors, title blocks
Other:
- note added: "A"
- note added: "Wiggle Spine board"

Commit message: Fixes for shield grounds and module numbering
Parts:
- renumbered MOD3 to MOD2, MOD5 to MOD3, MOD7 to MOD4, MOD2 to MOD5, MOD4 to MOD6, MOD6 to MOD7

Commit message: Schematic footprint and refdes work
Parts:
- MOD1, MOD2, MOD3, MOD4, MOD5, MOD6, MOD7: footprint (none) -> Socket_Strips:Socket_Strip_Angled_2x10
