File: boards/spine/spine-modules.sch (KiCad schematic (older format))
At the start: 7 parts

Commit message: BOM cleanup
Especially fix the confusing and mostly incorrect Mfg/Mfr stuff that I inherited from somewhere.
Parts:
- MOD1, MOD2, MOD3, MOD4, MOD5, MOD6, MOD7: Mfg1 (none) -> Centronic; Mfg1Id (none) -> 230-20; MfgId 230-20 -> (none); MfrId Centronic -> (none)
Changed lines of the file:
@@
 F 2 "Socket_Strips:Socket_Strip_Angled_2x10_Mirror" H 2650 1850 60  0001 C CNN
 F 3 "http://www.centronic.url.tw/pf/p29.pdf" H 2650 1850 60  0001 C CNN
-F 4 "Centronic" H 2650 3050 60  0001 C CNN "MfrId"
-F 5 "230-20" H 2650 3050 60  0001 C CNN "MfgId"
+F 4 "Centronic" H 2650 3050 60  0001 C CNN "Mfg1"
+F 5 "230-20" H 2650 3050 60  0001 C CNN "Mfg1Id"
 F 6 "eBay" H 2650 3050 60  0001 C CNN "Vend1"
 F 7 "http://www.ebay.com/itm/20pcs-2-54mm-pitch-2x10Pin-Header-Right-Angle-Female-Double-Row-Socket-Connector-/271560108036" H 2650 3050 60  0001 C CNN "Vend1Id"
@@
 F 2 "Socket_Strips:Socket_Strip_Angled_2x10_Mirror" H 4550 1850 60  0001 C CNN
 F 3 "http://www.centronic.url.tw/pf/p29.pdf" H 4550 1850 60  0001 C CNN
-F 4 "Centronic" H 4550 3050 60  0001 C CNN "MfrId"
-F 5 "230-20" H 4550 3050 60  0001 C CNN "MfgId"
+F 4 "Centronic" H 4550 3050 60  0001 C CNN "Mfg1"
+F 5 "230-20" H 4550 3050 60  0001 C CNN "Mfg1Id"
 F 6 "eBay" H 4550 3050 60  0001 C CNN "Vend1"
 F 7 "http://www.ebay.com/itm/20pcs-2-54mm-pitch-2x10Pin-Header-Right-Angle-Female-Double-Row-Socket-Connector-/271560108036" H 4550 3050 60  0001 C CNN "Vend1Id"
@@
 F 2 "Socket_Strips:Socket_Strip_Angled_2x10_Mirror" H 6450 1850 60  0001 C CNN
 F 3 "http://www.centronic.url.tw/pf/p29.pdf" H 6450 1850 60  0001 C CNN
-F 4 "Centronic" H 6450 3050 60  0001 C CNN "MfrId"
-F 5 "230-20" H 6450 3050 60  0001 C CNN "MfgId"
+F 4 "Centronic" H 6450 3050 60  0001 C CNN "Mfg1"
+F 5 "230-20" H 6450 3050 60  0001 C CNN "Mfg1Id"
 F 6 "eBay" H 6450 3050 60  0001 C CNN "Vend1"
 F 7 "http://www.ebay.com/itm/20pcs-2-54mm-pitch-2x10Pin-Header-Right-Angle-Female-Double-Row-Socket-Connector-/271560108036" H 6450 3050 60  0001 C CNN "Vend1Id"
@@
 F 2 "Socket_Strips:Socket_Strip_Angled_2x10_Mirror" H 8350 1850 60  0001 C CNN
 F 3 "http://www.centronic.url.tw/pf/p29.pdf" H 8350 1850 60  0001 C CNN
-F 4 "Centronic" H 8350 3050 60  0001 C CNN "MfrId"
-F 5 "230-20" H 8350 3050 60  0001 C CNN "MfgId"
+F 4 "Centronic" H 8350 3050 60  0001 C CNN "Mfg1"
+F 5 "230-20" H 8350 3050 60  0001 C CNN "Mfg1Id"
 F 6 "eBay" H 8350 3050 60  0001 C CNN "Vend1"
 F 7 "http://www.ebay.com/itm/20pcs-2-54mm-pitch-2x10Pin-Header-Right-Angle-Female-Double-Row-Socket-Connector-/271560108036" H 8350 3050 60  0001 C CNN "Vend1Id"
@@
 F 2 "Socket_Strips:Socket_Strip_Angled_2x10_Mirror" H 3600 3400 60  0001 C CNN
 F 3 "http://www.centronic.url.tw/pf/p29.pdf" H 3600 3400 60  0001 C CNN
-F 4 "Centronic" H 3600 4600 60  0001 C CNN "MfrId"
-F 5 "230-20" H 3600 4600 60  0001 C CNN "MfgId"
+F 4 "Centronic" H 3600 4600 60  0001 C CNN "Mfg1"
+F 5 "230-20" H 3600 4600 60  0001 C CNN "Mfg1Id"
 F 6 "eBay" H 3600 4600 60  0001 C CNN "Vend1"
 F 7 "http://www.ebay.com/itm/20pcs-2-54mm-pitch-2x10Pin-Header-Right-Angle-Female-Double-Row-Socket-Connector-/271560108036" H 3600 4600 60  0001 C CNN "Vend1Id"
@@
 F 2 "Socket_Strips:Socket_Strip_Angled_2x10_Mirror" H 5500 3400 60  0001 C CNN
 F 3 "http://www.centronic.url.tw/pf/p29.pdf" H 5500 3400 60  0001 C CNN
-F 4 "Centronic" H 5500 4600 60  0001 C CNN "MfrId"
-F 5 "230-20" H 5500 4600 60  0001 C CNN "MfgId"
+F 4 "Centronic" H 5500 4600 60  0001 C CNN "Mfg1"
+F 5 "230-20" H 5500 4600 60  0001 C CNN "Mfg1Id"
 F 6 "eBay" H 5500 4600 60  0001 C CNN "Vend1"
 F 7 "http://www.ebay.com/itm/20pcs-2-54mm-pitch-2x10Pin-Header-Right-Angle-Female-Double-Row-Socket-Connector-/271560108036" H 5500 4600 60  0001 C CNN "Vend1Id"
@@
 F 2 "Socket_Strips:Socket_Strip_Angled_2x10_Mirror" H 7400 3400 60  0001 C CNN
 F 3 "http://www.centronic.url.tw/pf/p29.pdf" H 7400 3400 60  0001 C CNN
-F 4 "Centronic" H 7400 4600 60  0001 C CNN "MfrId"
-F 5 "230-20" H 7400 4600 60  0001 C CNN "MfgId"
+F 4 "Centronic" H 7400 4600 60  0001 C CNN "Mfg1"
+F 5 "230-20" H 7400 4600 60  0001 C CNN "Mfg1Id"
 F 6 "eBay" H 7400 4600 60  0001 C CNN "Vend1"
 F 7 "http://www.ebay.com/itm/20pcs-2-54mm-pitch-2x10Pin-Header-Right-Angle-Female-Double-Row-Socket-Connector-/271560108036" H 7400 4600 60  0001 C CNN "Vend1Id"
@@
 72 0F 1C A9 DC 70 49 CB 79 33 88 85 99 AD 01 6C 4B 10 FC 3B 13 DE 3B 37 68 79 AD 07 BC 00 3C 0E
 3C 31 EE E3 D8 E7 0F 03 D7 7B 9F FB C1 E1 FF 01 18 C4 96 1D B8 0E 40 07 00 00 00 00 49 45 4E 44
-AE 42 60 82 00
+AE 42 60 82 44
 EndData
 $EndBitmap

Commit message: Capacitor upgrades, BOM tidying
Parts:
- renumbered MOD5 to MOD2, MOD2 to MOD3, MOD6 to MOD4, MOD3 to MOD5, MOD7 to MOD6, MOD4 to MOD7
