File: boards/spine/spine-modules.sch (KiCad schematic (older format))
At the start: 7 parts

Commit message: Redo component annotation
Noticed the module numbers were wrong after the last reannotation, so this seemed like a good time to reannotate again.
Parts:
- renumbered MOD3 to MOD2, MOD5 to MOD3, MOD7 to MOD4, MOD2 to MOD5, MOD4 to MOD6, MOD6 to MOD7
Changed lines of the file:
@@
 8x GPIOs per module (3.3V ONLY)\nLimited ESD protection (2kV HBM) on each I/O.\n\n3.3v and 5v supplied by system DC/DC converters.\nAt least 100mA available per module.\n\n24v rail is actually 5-24v, up to 4A per module.\n
 $Comp
-L CONN_02X10 MOD3
+L CONN_02X10 MOD2
 U 1 1 5641FA35
 P 4550 3050
-F 0 "MOD3" H 4550 3600 50  0000 C CNN
+F 0 "MOD2" H 4550 3600 50  0000 C CNN
 F 1 "2.54mm 2x10 right angle female header" V 4550 3050 50  0001 C CNN
 F 2 "Socket_Strips:Socket_Strip_Angled_2x10_Mirror" H 4550 1850 60  0001 C CNN
@@
 $EndComp
 $Comp
-L CONN_02X10 MOD5
+L CONN_02X10 MOD3
 U 1 1 5641FA76
 P 6450 3050
-F 0 "MOD5" H 6450 3600 50  0000 C CNN
+F 0 "MOD3" H 6450 3600 50  0000 C CNN
 F 1 "2.54mm 2x10 right angle female header" V 6450 3050 50  0001 C CNN
 F 2 "Socket_Strips:Socket_Strip_Angled_2x10_Mirror" H 6450 1850 60  0001 C CNN
@@
 $EndComp
 $Comp
-L CONN_02X10 MOD7
+L CONN_02X10 MOD4
 U 1 1 5641FAB5
 P 8350 3050
-F 0 "MOD7" H 8350 3600 50  0000 C CNN
+F 0 "MOD4" H 8350 3600 50  0000 C CNN
 F 1 "2.54mm 2x10 right angle female header" V 8350 3050 50  0001 C CNN
 F 2 "Socket_Strips:Socket_Strip_Angled_2x10_Mirror" H 8350 1850 60  0001 C CNN
@@
 $EndComp
 $Comp
-L CONN_02X10 MOD2
+L CONN_02X10 MOD5
 U 1 1 5641FAF2
 P 3600 4600
-F 0 "MOD2" H 3600 5150 50  0000 C CNN
+F 0 "MOD5" H 3600 5150 50  0000 C CNN
 F 1 "2.54mm 2x10 right angle female header" V 3600 4600 50  0001 C CNN
 F 2 "Socket_Strips:Socket_Strip_Angled_2x10_Mirror" H 3600 3400 60  0001 C CNN
@@
 $EndComp
 $Comp
-L CONN_02X10 MOD4
+L CONN_02X10 MOD6
 U 1 1 5641FB49
 P 5500 4600
-F 0 "MOD4" H 5500 5150 50  0000 C CNN
+F 0 "MOD6" H 5500 5150 50  0000 C CNN
 F 1 "2.54mm 2x10 right angle female header" V 5500 4600 50  0001 C CNN
 F 2 "Socket_Strips:Socket_Strip_Angled_2x10_Mirror" H 5500 3400 60  0001 C CNN
@@
 $EndComp
 $Comp
-L CONN_02X10 MOD6
+L CONN_02X10 MOD7
 U 1 1 5641FB8C
 P 7400 4600
-F 0 "MOD6" H 7400 5150 50  0000 C CNN
+F 0 "MOD7" H 7400 5150 50  0000 C CNN
 F 1 "2.54mm 2x10 right angle female header" V 7400 4600 50  0001 C CNN
 F 2 "Socket_Strips:Socket_Strip_Angled_2x10_Mirror" H 7400 3400 60  0001 C CNN
@@
 FB 59 00 E6 A5 69 3A 37 9E CF 73 BC F7 37 E3 33 5D 9E A8 3E 7F 80 FA F7 F6 BB 44 F4 6E D4 E7 77
 A2 1E 1F 27 A2 E3 16 70 32 E9 54 FE 3F E7 AF 00 CA 1C A3 36 0A 00 00 00 00 49 45 4E 44 AE 42 60
-82 00
+82 8F
 EndData
 $EndBitmap
@@
 72 0F 1C A9 DC 70 49 CB 79 33 88 85 99 AD 01 6C 4B 10 FC 3B 13 DE 3B 37 68 79 AD 07 BC 00 3C 0E
 3C 31 EE E3 D8 E7 0F 03 D7 7B 9F FB C1 E1 FF 01 18 C4 96 1D B8 0E 40 07 00 00 00 00 49 45 4E 44
-AE 42 60 82 11
+AE 42 60 82 00
 EndData
 $EndBitmap
