File: boards/spine/spine-usb.sch (KiCad schematic (older format))
At the start: 36 parts, among them CON5 USB-B, U1 93C56, U2 FT2232H, X2 12 MHz

Commit message: Simpler indicator LED strategy
Parts:
- C1: footprint TO_SOT_Packages_SMD:SOT-886 -> Capacitors_SMD:C_0805
- D1: footprint SOT363:SOT363 -> TO_SOT_Packages_SMD:SOT-23-6
Changed lines of the file:
@@
 F 0 "D1" H 1750 3550 50  0000 C CNN
 F 1 "TVS DIODE 5.5VWM" H 2250 2350 50  0001 C CNN
-F 2 "SOT363:SOT363" V 2700 3050 60  0001 C CNN
+F 2 "TO_SOT_Packages_SMD:SOT-23-6" V 2700 3050 60  0001 C CNN
 F 3 "http://www.nxp.com/documents/data_sheet/PRTR5V0U4Y.pdf" V 2700 3050 60  0001 C CNN
 F 4 "NXP" H 2250 3150 60  0001 C CNN "MfrId"
@@
 F 0 "C1" H 1050 5300 50  0000 L CNN
 F 1 "0.1uF" H 1050 5250 50  0000 L TNN
-F 2 "TO_SOT_Packages_SMD:SOT-886" H 1088 5250 30  0001 C CNN
+F 2 "Capacitors_SMD:C_0805" H 1088 5250 30  0001 C CNN
 F 3 "http://psearch.murata.com/capacitor/product/GRM21BR71H104MA01%23.pdf" H 1050 5400 60  0001 C CNN
 F 4 "0.01880" V 1050 5400 60  0001 C CNN "RefPrice1k"
@@
 72 0F 1C A9 DC 70 49 CB 79 33 88 85 99 AD 01 6C 4B 10 FC 3B 13 DE 3B 37 68 79 AD 07 BC 00 3C 0E
 3C 31 EE E3 D8 E7 0F 03 D7 7B 9F FB C1 E1 FF 01 18 C4 96 1D B8 0E 40 07 00 00 00 00 49 45 4E 44
-AE 42 60 82 00
+AE 42 60 82 A3
 EndData
 $EndBitmap

Commit message: Fix some 6-pin packages
I had several of these mislabeled as SOT23-6, but there are no SOT23-6 parts here. The LDOs are SOT23-5, and the others (TVS diode array and inverters) are in the smaller SC-88 package.
Parts:
- D1: footprint TO_SOT_Packages_SMD:SOT-23-6 -> TO_SOT_Packages_SMD:SC-70-6
Changed lines of the file:
@@
 $EndComp
 $Comp
-L GND #PWR4
+L GND #PWR01
 U 1 1 563F3C00
 P 1500 4000
-F 0 "#PWR4" H 1500 3750 50  0001 C CNN
+F 0 "#PWR01" H 1500 3750 50  0001 C CNN
 F 1 "GND" H 1500 3850 50  0000 C CNN
 F 2 "" H 1500 4000 60  0000 C CNN
@@
 $EndComp
 $Comp
-L +3V3 #PWR12
+L +3V3 #PWR02
 U 1 1 563F5B33
 P 4500 1350
-F 0 "#PWR12" H 4500 1200 50  0001 C CNN
+F 0 "#PWR02" H 4500 1200 50  0001 C CNN
 F 1 "+3V3" H 4500 1490 50  0000 C CNN
 F 2 "" H 4500 1350 60  0000 C CNN
@@
 F 0 "D1" H 1750 3550 50  0000 C CNN
 F 1 "TVS DIODE 5.5VWM" H 2250 2350 50  0001 C CNN
-F 2 "TO_SOT_Packages_SMD:SOT-23-6" V 2700 3050 60  0001 C CNN
+F 2 "TO_SOT_Packages_SMD:SC-70-6" V 2700 3050 60  0001 C CNN
 F 3 "http://www.nxp.com/documents/data_sheet/PRTR5V0U4Y.pdf" V 2700 3050 60  0001 C CNN
 F 4 "NXP" H 2250 3150 60  0001 C CNN "MfrId"
@@
 NoConn ~ 1950 3800
 $Comp
-L GND #PWR13
+L GND #PWR03
 U 1 1 56407FC9
 P 4500 3550
-F 0 "#PWR13" H 4500 3300 50  0001 C CNN
+F 0 "#PWR03" H 4500 3300 50  0001 C CNN
 F 1 "GND" H 4500 3400 50  0000 C CNN
 F 2 "" H 4500 3550 60  0000 C CNN
@@
 $EndComp
 $Comp
-L +3V3 #PWR17
+L +3V3 #PWR04
 U 1 1 56409B2C
 P 7350 950
-F 0 "#PWR17" H 7350 800 50  0001 C CNN
+F 0 "#PWR04" H 7350 800 50  0001 C CNN
 F 1 "+3V3" H 7350 1090 50  0000 C CNN
 F 2 "" H 7350 950 60  0000 C CNN
@@
 $EndComp
 $Comp
-L +3V3 #PWR2
+L +3V3 #PWR05
 U 1 1 5640C498
 P 1050 5000
-F 0 "#PWR2" H 1050 4850 50  0001 C CNN
+F 0 "#PWR05" H 1050 4850 50  0001 C CNN
 F 1 "+3V3" H 1050 5140 50  0000 C CNN
 F 2 "" H 1050 5000 60  0000 C CNN
@@
 $EndComp
 $Comp
-L GND #PWR3
+L GND #PWR06
 U 1 1 5640C700
 P 1050 5800
-F 0 "#PWR3" H 1050 5550 50  0001 C CNN
+F 0 "#PWR06" H 1050 5550 50  0001 C CNN
 F 1 "GND" H 1050 5650 50  0000 C CNN
 F 2 "" H 1050 5800 60  0000 C CNN
@@
 $EndComp
 $Comp
-L +3V3 #PWR6
+L +3V3 #PWR07
 U 1 1 5640CB0D
 P 2800 4500
-F 0 "#PWR6" H 2800 4350 50  0001 C CNN
+F 0 "#PWR07" H 2800 4350 50  0001 C CNN
 F 1 "+3V3" H 2800 4640 50  0000 C CNN
 F 2 "" H 2800 4500 60  0000 C CNN
@@
 $EndComp
 $Comp
-L GND #PWR5
+L GND #PWR08
 U 1 1 5640EC58
 P 1750 7450
-F 0 "#PWR5" H 1750 7200 50  0001 C CNN
+F 0 "#PWR08" H 1750 7200 50  0001 C CNN
 F 1 "GND" H 1750 7300 50  0000 C CNN
 F 2 "" H 1750 7450 60  0000 C CNN
@@
 $EndComp
 $Comp
-L GND #PWR8
+L GND #PWR09
 U 1 1 5640ECEA
 P 2900 1650
-F 0 "#PWR8" H 2900 1400 50  0001 C CNN
+F 0 "#PWR09" H 2900 1400 50  0001 C CNN
 F 1 "GND" H 2900 1500 50  0000 C CNN
 F 2 "" H 2900 1650 60  0000 C CNN
@@
 FTDI_1V8REG
 $Comp
-L +3V3 #PWR7
+L +3V3 #PWR010
 U 1 1 5640F443
 P 2900 1000
-F 0 "#PWR7" H 2900 850 50  0001 C CNN
+F 0 "#PWR010" H 2900 850 50  0001 C CNN
 F 1 "+3V3" H 2900 1140 50  0000 C CNN
 F 2 "" H 2900 1000 60  0000 C CNN
@@
 $EndComp
 $Comp
-L GND #PWR11
+L GND #PWR011
 U 1 1 56411C34
 P 4450 5800
-F 0 "#PWR11" H 4450 5550 50  0001 C CNN
+F 0 "#PWR011" H 4450 5550 50  0001 C CNN
 F 1 "GND" H 4450 5650 50  0000 C CNN
 F 2 "" H 4450 5800 60  0000 C CNN
@@
 $EndComp
 $Comp
-L GND #PWR16
+L GND #PWR012
 U 1 1 56412014
 P 6450 5800
-F 0 "#PWR16" H 6450 5550 50  0001 C CNN
+F 0 "#PWR012" H 6450 5550 50  0001 C CNN
 F 1 "GND" H 6450 5650 50  0000 C CNN
 F 2 "" H 6450 5800 60  0000 C CNN
@@
 $EndComp
 $Comp
-L GND #PWR10
+L GND #PWR013
 U 1 1 5642A93B
 P 3400 7450
-F 0 "#PWR10" H 3400 7200 50  0001 C CNN
+F 0 "#PWR013" H 3400 7200 50  0001 C CNN
 F 1 "GND" H 3400 7300 50  0000 C CNN
 F 2 "" H 3400 7450 60  0000 C CNN
@@
 	3700 7400 3700 7300
 $Comp
-L +3V3 #PWR9
+L +3V3 #PWR014
 U 1 1 5642B955
 P 3400 6450
-F 0 "#PWR9" H 3400 6300 50  0001 C CNN
+F 0 "#PWR014" H 3400 6300 50  0001 C CNN
 F 1 "+3V3" H 3400 6590 50  0000 C CNN
 F 2 "" H 3400 6450 60  0000 C CNN
@@
 $EndComp
 $Comp
-L GND #PWR15
+L GND #PWR015
 U 1 1 5642BC5C
 P 4750 7450
-F 0 "#PWR15" H 4750 7200 50  0001 C CNN
+F 0 "#PWR015" H 4750 7200 50  0001 C CNN
 F 1 "GND" H 4750 7300 50  0000 C CNN
 F 2 "" H 4750 7450 60  0000 C CNN
@@
 	5050 7400 5050 7300
 $Comp
-L +3V3 #PWR14
+L +3V3 #PWR016
 U 1 1 5642BC76
 P 4750 6450
-F 0 "#PWR14" H 4750 6300 50  0001 C CNN
+F 0 "#PWR016" H 4750 6300 50  0001 C CNN
 F 1 "+3V3" H 4750 6590 50  0000 C CNN
 F 2 "" H 4750 6450 60  0000 C CNN
@@
 72 0F 1C A9 DC 70 49 CB 79 33 88 85 99 AD 01 6C 4B 10 FC 3B 13 DE 3B 37 68 79 AD 07 BC 00 3C 0E
 3C 31 EE E3 D8 E7 0F 03 D7 7B 9F FB C1 E1 FF 01 18 C4 96 1D B8 0E 40 07 00 00 00 00 49 45 4E 44
-AE 42 60 82 A3
+AE 42 60 82 00
 EndData
 $EndBitmap
@@
 	1500 3900 3450 3900
 $Comp
-L Earth #PWR1
+L Earth #PWR017
 U 1 1 565B7DB6
 P 1050 2850
-F 0 "#PWR1" H 1050 2600 50  0001 C CNN
+F 0 "#PWR017" H 1050 2600 50  0001 C CNN
 F 1 "Earth" H 1050 2700 50  0001 C CNN
 F 2 "" H 1050 2850 60  0000 C CNN

Commit message: Switch to a ferrite bead with 6A current rating
Parts:
- FB1, FB2, FB3, FB4: MfgId CIB21P260NE -> CIS21P300NE; RefPrice1k 0.00906 -> 0.02383; Vend1Id 1276-6342-2-ND -> 1276-6370-1-ND
Changed lines of the file:
@@
 F 1 "Ferrite bead" H 2000 2400 39  0001 C BNN
 F 2 "Resistors_SMD:R_0805" H 1600 2500 50  0001 C CNN
-F 3 "http://www.samsungsem.com/kr/front/downloadcms.do?path=/kr/support/product-search/bead/__icsFiles/afieldfile/2014/11/13&fileName=S_CIB21P110NE.pdf" H 1625 2350 60  0001 C CNN
-F 4 "0.00906" H 1600 2350 60  0001 C CNN "RefPrice1k"
+F 3 "http://www.samsungsem.com/kr/front/downloadcms.do?path=/kr/support/product-search/bead/__icsFiles/afieldfile/2014/11/13&fileName=S_CIS21J121NE.pdf" H 1625 2350 60  0001 C CNN
+F 4 "0.02383" H 1600 2350 60  0001 C CNN "RefPrice1k"
 F 5 "Samsung" H 1600 2350 60  0001 C CNN "MfrId"
-F 6 "CIB21P260NE" H 1600 2350 60  0001 C CNN "MfgId"
+F 6 "CIS21P300NE" H 1600 2350 60  0001 C CNN "MfgId"
 F 7 "Digikey" H 1600 2350 60  0001 C CNN "Vend1"
-F 8 "1276-6342-2-ND" H 1600 2350 60  0001 C CNN "Vend1Id"
+F 8 "1276-6370-1-ND" H 1600 2350 60  0001 C CNN "Vend1Id"
 	1    1600 2350
 	1    0    0    -1
@@
 F 1 "Ferrite bead" H 1900 3050 39  0001 C BNN
 F 2 "Resistors_SMD:R_0805" H 1500 3300 50  0001 C CNN
-F 3 "http://www.samsungsem.com/kr/front/downloadcms.do?path=/kr/support/product-search/bead/__icsFiles/afieldfile/2014/11/13&fileName=S_CIB21P110NE.pdf" H 1525 3150 60  0001 C CNN
-F 4 "0.00906" H 1500 3150 60  0001 C CNN "RefPrice1k"
+F 3 "http://www.samsungsem.com/kr/front/downloadcms.do?path=/kr/support/product-search/bead/__icsFiles/afieldfile/2014/11/13&fileName=S_CIS21J121NE.pdf" H 1525 3150 60  0001 C CNN
+F 4 "0.02383" H 1500 3150 60  0001 C CNN "RefPrice1k"
 F 5 "Samsung" H 1500 3150 60  0001 C CNN "MfrId"
-F 6 "CIB21P260NE" H 1500 3150 60  0001 C CNN "MfgId"
+F 6 "CIS21P300NE" H 1500 3150 60  0001 C CNN "MfgId"
 F 7 "Digikey" H 1500 3150 60  0001 C CNN "Vend1"
-F 8 "1276-6342-2-ND" H 1500 3150 60  0001 C CNN "Vend1Id"
+F 8 "1276-6370-1-ND" H 1500 3150 60  0001 C CNN "Vend1Id"
 	1    1500 3150
 	0    -1   -1   0
@@
 F 1 "Ferrite bead" H 3800 6500 39  0001 C BNN
 F 2 "Resistors_SMD:R_0805" H 3400 6600 50  0001 C CNN
-F 3 "http://www.samsungsem.com/kr/front/downloadcms.do?path=/kr/support/product-search/bead/__icsFiles/afieldfile/2014/11/13&fileName=S_CIB21P110NE.pdf" H 3425 6450 60  0001 C CNN
-F 4 "0.00906" H 3400 6450 60  0001 C CNN "RefPrice1k"
+F 3 "http://www.samsungsem.com/kr/front/downloadcms.do?path=/kr/support/product-search/bead/__icsFiles/afieldfile/2014/11/13&fileName=S_CIS21J121NE.pdf" H 3425 6450 60  0001 C CNN
+F 4 "0.02383" H 3400 6450 60  0001 C CNN "RefPrice1k"
 F 5 "Samsung" H 3400 6450 60  0001 C CNN "MfrId"
-F 6 "CIB21P260NE" H 3400 6450 60  0001 C CNN "MfgId"
+F 6 "CIS21P300NE" H 3400 6450 60  0001 C CNN "MfgId"
 F 7 "Digikey" H 3400 6450 60  0001 C CNN "Vend1"
-F 8 "1276-6342-2-ND" H 3400 6450 60  0001 C CNN "Vend1Id"
+F 8 "1276-6370-1-ND" H 3400 6450 60  0001 C CNN "Vend1Id"
 	1    3400 6450
 	0    1    1    0
@@
 F 1 "Ferrite bead" H 5150 6500 39  0001 C BNN
 F 2 "Resistors_SMD:R_0805" H 4750 6600 50  0001 C CNN
-F 3 "http://www.samsungsem.com/kr/front/downloadcms.do?path=/kr/support/product-search/bead/__icsFiles/afieldfile/2014/11/13&fileName=S_CIB21P110NE.pdf" H 4775 6450 60  0001 C CNN
-F 4 "0.00906" H 4750 6450 60  0001 C CNN "RefPrice1k"
+F 3 "http://www.samsungsem.com/kr/front/downloadcms.do?path=/kr/support/product-search/bead/__icsFiles/afieldfile/2014/11/13&fileName=S_CIS21J121NE.pdf" H 4775 6450 60  0001 C CNN
+F 4 "0.02383" H 4750 6450 60  0001 C CNN "RefPrice1k"
 F 5 "Samsung" H 4750 6450 60  0001 C CNN "MfrId"
-F 6 "CIB21P260NE" H 4750 6450 60  0001 C CNN "MfgId"
+F 6 "CIS21P300NE" H 4750 6450 60  0001 C CNN "MfgId"
 F 7 "Digikey" H 4750 6450 60  0001 C CNN "Vend1"
-F 8 "1276-6342-2-ND" H 4750 6450 60  0001 C CNN "Vend1Id"
+F 8 "1276-6370-1-ND" H 4750 6450 60  0001 C CNN "Vend1Id"
 	1    4750 6450
 	0    1    1    0
