File: boards/spine/spine-usb.sch (KiCad schematic (older format))
At the start: 36 parts, among them CON5 USB-B, U1 93C56, U2 FT2232H, X2 12 MHz

Commit message: BOM cleanup
Especially fix the confusing and mostly incorrect Mfg/Mfr stuff that I inherited from somewhere.
Parts:
- C1, C11, C14, C2, C3, C4, C5, C6, C7, C8, C9: Mfg1 (none) -> Murata; Mfg1Id (none) -> GRM21BR71H104MA01L; MfgId GRM21BR71H104MA01L -> (none); MfrId Murata -> (none)
- C10, C13, C15, C17: Mfg1 (none) -> Murata; Mfg1Id (none) -> GRM31CR61H106MA12L; MfgId GRM31CR61H106MA12L -> (none); MfrId Murata -> (none)
- C12, C16: Mfg1 (none) -> Samsung; Mfg1Id (none) -> CL21C200JBANNNC; MfgId CL21C200JBANNNC -> (none); MfrId Samsung -> (none)
- CON5: Mfg1 (none) -> Pulse; Mfg1Id (none) -> E8144-B02022-L; MfgId E8144-B02022-L -> (none); MfrId Pulse -> (none)
- D1: Mfg1 (none) -> NXP; Mfg1Id (none) -> PRTR5V0U4Y; MfgId PRTR5V0U4Y -> (none); MfrId NXP -> (none)
- FB1, FB2, FB3, FB4: Mfg1 (none) -> Samsung; Mfg1Id (none) -> CIS21P300NE; MfgId CIS21P300NE -> (none); MfrId Samsung -> (none)
- R1, R2, R3, R5: Mfg1 (none) -> Stackpole; Mfg1Id (none) -> RMCF0805JT10K0; MfgId RMCF0805JT10K0 -> (none); MfrId Stackpole -> (none)
- R10: Mfg1 (none) -> Stackpole; Mfg1Id (none) -> RMCF0805FT12K0; MfgId RMCF0805FT12K0 -> (none); MfrId Stackpole -> (none)
- R4, R7: Mfg1 (none) -> Stackpole; Mfg1Id (none) -> RMCF0805JT4K70; MfgId RMCF0805JT4K70 -> (none); MfrId Stackpole -> (none)
- R6: Mfg1 (none) -> Stackpole; Mfg1Id (none) -> RMCF0805JT2K20CT; MfgId RMCF0805JT2K20CT -> (none); MfrId Stackpole -> (none)
- R8, R9: Mfg1 (none) -> Stackpole; Mfg1Id (none) -> RMCF0805JT10R0CT; MfgId RMCF0805JT10R0CT -> (none); MfrId Stackpole -> (none)
- U1: Mfg1 (none) -> ON Semi; Mfg1Id (none) -> CAT93C56VI-GT3; MfgId CAT93C56VI-GT3 -> (none); MfrId ON Semi -> (none)
- U2: Mfg1 (none) -> FTDI; Mfg1Id (none) -> FT2232HL-REEL; MfgId FT2232HL-REEL -> (none); MfrId FTDI -> (none)
- X2: Mfg1 (none) -> Abracon; Mfg1Id (none) -> ABLS-12.000MHZ-B4-T; MfgId ABLS-12.000MHZ-B4-T -> (none); MfrId Abracon -> (none)

Commit message: Capacitor upgrades, BOM tidying
Parts:
- renumbered CON5 to CON1, X2 to X1
Changed lines of the file:
@@
 $EndDescr
 $Comp
-L USB_B CON5
+L USB_B CON1
 U 1 1 5637E4EA
 P 1150 2550
-F 0 "CON5" V 850 2650 50  0000 C CNN
+F 0 "CON1" V 850 2650 50  0000 C CNN
 F 1 "USB-B" H 1100 2750 50  0000 C CNN
 F 2 "Connect:USB_B" V 1100 2450 60  0001 C CNN
@@
 $EndComp
 $Comp
-L GND #PWR01
+L GND #PWR4
 U 1 1 563F3C00
 P 1500 4000
-F 0 "#PWR01" H 1500 3750 50  0001 C CNN
+F 0 "#PWR4" H 1500 3750 50  0001 C CNN
 F 1 "GND" H 1500 3850 50  0000 C CNN
 F 2 "" H 1500 4000 60  0000 C CNN
@@
 $EndComp
 $Comp
-L +3V3 #PWR02
+L +3V3 #PWR12
 U 1 1 563F5B33
 P 4500 1350
-F 0 "#PWR02" H 4500 1200 50  0001 C CNN
+F 0 "#PWR12" H 4500 1200 50  0001 C CNN
 F 1 "+3V3" H 4500 1490 50  0000 C CNN
 F 2 "" H 4500 1350 60  0000 C CNN
@@
 NoConn ~ 1950 3800
 $Comp
-L GND #PWR03
+L GND #PWR13
 U 1 1 56407FC9
 P 4500 3550
-F 0 "#PWR03" H 4500 3300 50  0001 C CNN
+F 0 "#PWR13" H 4500 3300 50  0001 C CNN
 F 1 "GND" H 4500 3400 50  0000 C CNN
 F 2 "" H 4500 3550 60  0000 C CNN
@@
 $EndComp
 $Comp
-L +3V3 #PWR04
+L +3V3 #PWR17
 U 1 1 56409B2C
 P 7350 950
-F 0 "#PWR04" H 7350 800 50  0001 C CNN
+F 0 "#PWR17" H 7350 800 50  0001 C CNN
 F 1 "+3V3" H 7350 1090 50  0000 C CNN
 F 2 "" H 7350 950 60  0000 C CNN
@@
 $EndComp
 $Comp
-L +3V3 #PWR05
+L +3V3 #PWR2
 U 1 1 5640C498
 P 1050 5000
-F 0 "#PWR05" H 1050 4850 50  0001 C CNN
+F 0 "#PWR2" H 1050 4850 50  0001 C CNN
 F 1 "+3V3" H 1050 5140 50  0000 C CNN
 F 2 "" H 1050 5000 60  0000 C CNN
@@
 $EndComp
 $Comp
-L GND #PWR06
+L GND #PWR3
 U 1 1 5640C700
 P 1050 5800
-F 0 "#PWR06" H 1050 5550 50  0001 C CNN
+F 0 "#PWR3" H 1050 5550 50  0001 C CNN
 F 1 "GND" H 1050 5650 50  0000 C CNN
 F 2 "" H 1050 5800 60  0000 C CNN
@@
 $EndComp
 $Comp
-L +3V3 #PWR07
+L +3V3 #PWR6
 U 1 1 5640CB0D
 P 2800 4500
-F 0 "#PWR07" H 2800 4350 50  0001 C CNN
+F 0 "#PWR6" H 2800 4350 50  0001 C CNN
 F 1 "+3V3" H 2800 4640 50  0000 C CNN
 F 2 "" H 2800 4500 60  0000 C CNN
@@
 $EndComp
 $Comp
-L GND #PWR08
+L GND #PWR5
 U 1 1 5640EC58
 P 1750 7450
-F 0 "#PWR08" H 1750 7200 50  0001 C CNN
+F 0 "#PWR5" H 1750 7200 50  0001 C CNN
 F 1 "GND" H 1750 7300 50  0000 C CNN
 F 2 "" H 1750 7450 60  0000 C CNN
@@
 $EndComp
 $Comp
-L GND #PWR09
+L GND #PWR8
 U 1 1 5640ECEA
 P 2900 1650
-F 0 "#PWR09" H 2900 1400 50  0001 C CNN
+F 0 "#PWR8" H 2900 1400 50  0001 C CNN
 F 1 "GND" H 2900 1500 50  0000 C CNN
 F 2 "" H 2900 1650 60  0000 C CNN
@@
 FTDI_1V8REG
 $Comp
-L +3V3 #PWR010
+L +3V3 #PWR7
 U 1 1 5640F443
 P 2900 1000
-F 0 "#PWR010" H 2900 850 50  0001 C CNN
+F 0 "#PWR7" H 2900 850 50  0001 C CNN
 F 1 "+3V3" H 2900 1140 50  0000 C CNN
 F 2 "" H 2900 1000 60  0000 C CNN
@@
 NoConn ~ 8050 5150
 $Comp
-L Crystal X2
+L Crystal X1
 U 1 1 564105F5
 P 4750 4950
-F 0 "X2" H 4750 5100 50  0000 C CNN
+F 0 "X1" H 4750 5100 50  0000 C CNN
 F 1 "12 MHz" H 4750 4800 50  0000 C CNN
 F 2 "Crystals:Crystal_HC49-SD_SMD" H 4750 4950 60  0001 C CNN
@@
 $EndComp
 $Comp
-L GND #PWR011
+L GND #PWR11
 U 1 1 56411C34
 P 4450 5800
-F 0 "#PWR011" H 4450 5550 50  0001 C CNN
+F 0 "#PWR11" H 4450 5550 50  0001 C CNN
 F 1 "GND" H 4450 5650 50  0000 C CNN
 F 2 "" H 4450 5800 60  0000 C CNN
@@
 $EndComp
 $Comp
-L GND #PWR012
+L GND #PWR16
 U 1 1 56412014
 P 6450 5800
-F 0 "#PWR012" H 6450 5550 50  0001 C CNN
+F 0 "#PWR16" H 6450 5550 50  0001 C CNN
 F 1 "GND" H 6450 5650 50  0000 C CNN
 F 2 "" H 6450 5800 60  0000 C CNN
@@
 $EndComp
 $Comp
-L GND #PWR013
+L GND #PWR10
 U 1 1 5642A93B
 P 3400 7450
-F 0 "#PWR013" H 3400 7200 50  0001 C CNN
+F 0 "#PWR10" H 3400 7200 50  0001 C CNN
 F 1 "GND" H 3400 7300 50  0000 C CNN
 F 2 "" H 3400 7450 60  0000 C CNN
@@
 	3700 7400 3700 7300
 $Comp
-L +3V3 #PWR014
+L +3V3 #PWR9
 U 1 1 5642B955
 P 3400 6450
-F 0 "#PWR014" H 3400 6300 50  0001 C CNN
+F 0 "#PWR9" H 3400 6300 50  0001 C CNN
 F 1 "+3V3" H 3400 6590 50  0000 C CNN
 F 2 "" H 3400 6450 60  0000 C CNN
@@
 $EndComp
 $Comp
-L GND #PWR015
+L GND #PWR15
 U 1 1 5642BC5C
 P 4750 7450
-F 0 "#PWR015" H 4750 7200 50  0001 C CNN
+F 0 "#PWR15" H 4750 7200 50  0001 C CNN
 F 1 "GND" H 4750 7300 50  0000 C CNN
 F 2 "" H 4750 7450 60  0000 C CNN
@@
 	5050 7400 5050 7300
 $Comp
-L +3V3 #PWR016
+L +3V3 #PWR14
 U 1 1 5642BC76
 P 4750 6450
-F 0 "#PWR016" H 4750 6300 50  0001 C CNN
+F 0 "#PWR14" H 4750 6300 50  0001 C CNN
 F 1 "+3V3" H 4750 6590 50  0000 C CNN
 F 2 "" H 4750 6450 60  0000 C CNN
@@
 FB 59 00 E6 A5 69 3A 37 9E CF 73 BC F7 37 E3 33 5D 9E A8 3E 7F 80 FA F7 F6 BB 44 F4 6E D4 E7 77
 A2 1E 1F 27 A2 E3 16 70 32 E9 54 FE 3F E7 AF 00 CA 1C A3 36 0A 00 00 00 00 49 45 4E 44 AE 42 60
-82 39
+82 00
 EndData
 $EndBitmap
@@
 72 0F 1C A9 DC 70 49 CB 79 33 88 85 99 AD 01 6C 4B 10 FC 3B 13 DE 3B 37 68 79 AD 07 BC 00 3C 0E
 3C 31 EE E3 D8 E7 0F 03 D7 7B 9F FB C1 E1 FF 01 18 C4 96 1D B8 0E 40 07 00 00 00 00 49 45 4E 44
-AE 42 60 82 FF
+AE 42 60 82 00
 EndData
 $EndBitmap
@@
 	1500 3900 3450 3900
 $Comp
-L Earth #PWR017
+L Earth #PWR1
 U 1 1 565B7DB6
 P 1050 2850
-F 0 "#PWR017" H 1050 2600 50  0001 C CNN
+F 0 "#PWR1" H 1050 2600 50  0001 C CNN
 F 1 "Earth" H 1050 2700 50  0001 C CNN
 F 2 "" H 1050 2850 60  0000 C CNN
