File: boards/spine/power-24v.sch (KiCad schematic (older format))
At the start: 9 parts, among them CON1 5-24V 5A, CON2 5-24V 16A, Q4 AOD4189

Commit message: Switch to a ferrite bead with 6A current rating
Parts:
- FB8, FB9: MfgId CIB21P260NE -> CIS21P300NE; RefPrice1k 0.00906 -> 0.02383; Vend1Id 1276-6342-2-ND -> 1276-6370-1-ND
Changed lines of the file:
@@
 F 1 "Ferrite bead" H 7500 4750 39  0001 C BNN
 F 2 "Resistors_SMD:R_0805" H 7100 5000 50  0001 C CNN
-F 3 "http://www.samsungsem.com/kr/front/downloadcms.do?path=/kr/support/product-search/bead/__icsFiles/afieldfile/2014/11/13&fileName=S_CIB21P110NE.pdf" H 7125 4850 60  0001 C CNN
-F 4 "0.00906" H 7100 4850 60  0001 C CNN "RefPrice1k"
+F 3 "http://www.samsungsem.com/kr/front/downloadcms.do?path=/kr/support/product-search/bead/__icsFiles/afieldfile/2014/11/13&fileName=S_CIS21J121NE.pdf" H 7125 4850 60  0001 C CNN
+F 4 "0.02383" H 7100 4850 60  0001 C CNN "RefPrice1k"
 F 5 "Samsung" H 7100 4850 60  0001 C CNN "MfrId"
-F 6 "CIB21P260NE" H 7100 4850 60  0001 C CNN "MfgId"
+F 6 "CIS21P300NE" H 7100 4850 60  0001 C CNN "MfgId"
 F 7 "Digikey" H 7100 4850 60  0001 C CNN "Vend1"
-F 8 "1276-6342-2-ND" H 7100 4850 60  0001 C CNN "Vend1Id"
+F 8 "1276-6370-1-ND" H 7100 4850 60  0001 C CNN "Vend1Id"
 	1    7100 4850
 	1    0    0    -1
@@
 F 1 "Ferrite bead" H 7500 5050 39  0001 C BNN
 F 2 "Resistors_SMD:R_0805" H 7100 5300 50  0001 C CNN
-F 3 "http://www.samsungsem.com/kr/front/downloadcms.do?path=/kr/support/product-search/bead/__icsFiles/afieldfile/2014/11/13&fileName=S_CIB21P110NE.pdf" H 7125 5150 60  0001 C CNN
-F 4 "0.00906" H 7100 5150 60  0001 C CNN "RefPrice1k"
+F 3 "http://www.samsungsem.com/kr/front/downloadcms.do?path=/kr/support/product-search/bead/__icsFiles/afieldfile/2014/11/13&fileName=S_CIS21J121NE.pdf" H 7125 5150 60  0001 C CNN
+F 4 "0.02383" H 7100 5150 60  0001 C CNN "RefPrice1k"
 F 5 "Samsung" H 7100 5150 60  0001 C CNN "MfrId"
-F 6 "CIB21P260NE" H 7100 5150 60  0001 C CNN "MfgId"
+F 6 "CIS21P300NE" H 7100 5150 60  0001 C CNN "MfgId"
 F 7 "Digikey" H 7100 5150 60  0001 C CNN "Vend1"
-F 8 "1276-6342-2-ND" H 7100 5150 60  0001 C CNN "Vend1Id"
+F 8 "1276-6370-1-ND" H 7100 5150 60  0001 C CNN "Vend1Id"
 	1    7100 5150
 	1    0    0    -1
