File: boards/spine/spine-sync.sch (KiCad schematic (older format))
At the start: 6 parts, among them CON3 PLR135, CON4 PLT133

Commit message: More simplification and BOM optimization
Thanks for the hints on the ST485 and dual-FETs, @mikelectricstuf!
Parts:
- CON3: MfgId Everlight -> PLR135/T10; MfrId PLR135/T10 -> Everlight
- CON4: MfgId Everlight -> PLT133/T; MfrId PLT133/T -> Everlight
Changed lines of the file:
@@
 F 4 "Digikey" H 5900 3100 60  0001 C CNN "Vend1"
 F 5 "1080-1428-ND" H 5900 3100 60  0001 C CNN "Vend1Id"
-F 6 "Everlight" H 5900 3100 60  0001 C CNN "MfgId"
-F 7 "PLT133/T" H 5900 3100 60  0001 C CNN "MfrId"
+F 6 "Everlight" H 5900 3100 60  0001 C CNN "MfrId"
+F 7 "PLT133/T" H 5900 3100 60  0001 C CNN "MfgId"
 F 8 "0.37125" H 5900 3100 60  0001 C CNN "RefPrice1k"
 	1    5900 3100
@@
 $EndComp
 $Comp
-L GND #PWR160
+L GND #PWR0159
 U 1 1 5650C9B4
 P 4750 3500
-F 0 "#PWR160" H 4750 3250 50  0001 C CNN
+F 0 "#PWR0159" H 4750 3250 50  0001 C CNN
 F 1 "GND" H 4750 3350 50  0000 C CNN
 F 2 "" H 4750 3500 60  0000 C CNN
@@
 $EndComp
 $Comp
-L +5V #PWR159
+L +5V #PWR0160
 U 1 1 5650C9FA
 P 4750 2700
-F 0 "#PWR159" H 4750 2550 50  0001 C CNN
+F 0 "#PWR0160" H 4750 2550 50  0001 C CNN
 F 1 "+5V" H 4750 2840 50  0000 C CNN
 F 2 "" H 4750 2700 60  0000 C CNN
@@
 F 5 "1080-1433-ND" H 4800 5100 60  0001 C CNN "Vend1Id"
 F 6 "0.73054" H 4800 5100 60  0001 C CNN "RefPrice1k"
-F 7 "Everlight" H 4800 5100 60  0001 C CNN "MfgId"
-F 8 "PLR135/T10" H 4800 5100 60  0001 C CNN "MfrId"
+F 7 "Everlight" H 4800 5100 60  0001 C CNN "MfrId"
+F 8 "PLR135/T10" H 4800 5100 60  0001 C CNN "MfgId"
 	1    4800 5100
 	1    0    0    -1
 $EndComp
 $Comp
-L +3.3V #PWR161
+L +3.3V #PWR0161
 U 1 1 5650E21A
 P 6050 4300
-F 0 "#PWR161" H 6050 4150 50  0001 C CNN
+F 0 "#PWR0161" H 6050 4150 50  0001 C CNN
 F 1 "+3.3V" H 6050 4440 50  0000 C CNN
 F 2 "" H 6050 4300 60  0000 C CNN
@@
 $EndComp
 $Comp
-L GND #PWR162
+L GND #PWR0162
 U 1 1 5650E275
 P 6050 5500
-F 0 "#PWR162" H 6050 5250 50  0001 C CNN
+F 0 "#PWR0162" H 6050 5250 50  0001 C CNN
 F 1 "GND" H 6050 5350 50  0000 C CNN
 F 2 "" H 6050 5500 60  0000 C CNN
@@
 FB 59 00 E6 A5 69 3A 37 9E CF 73 BC F7 37 E3 33 5D 9E A8 3E 7F 80 FA F7 F6 BB 44 F4 6E D4 E7 77
 A2 1E 1F 27 A2 E3 16 70 32 E9 54 FE 3F E7 AF 00 CA 1C A3 36 0A 00 00 00 00 49 45 4E 44 AE 42 60
-82 C1
+82 4F
 EndData
 $EndBitmap
