File: boards/spine/power-ldo.sch (KiCad schematic (older format))
At the start: 6 parts, among them U13 TCR2EF25, U14 TCR2EF12

Commit message: BOM cleanup
Especially fix the confusing and mostly incorrect Mfg/Mfr stuff that I inherited from somewhere.
Parts:
- C74, C76: Mfg1 (none) -> Murata; Mfg1Id (none) -> GRM21BR71H104MA01L; MfgId GRM21BR71H104MA01L -> (none); MfrId Murata -> (none)
- C75, C77: Mfg1 (none) -> Murata; Mfg1Id (none) -> GRM219R61H105KA73D; MfgId GRM219R61H105KA73D -> (none); MfrId Murata -> (none)
- U13: Mfg1 (none) -> Toshiba; Mfg1Id (none) -> TCR2EF25.LM(CT; MfgId TCR2EF25.LM(CT -> (none); MfrId Toshiba -> (none)
- U14: Mfg1 (none) -> Toshiba; Mfg1Id (none) -> TCR2EF12.LM(CT; MfgId TCR2EF12.LM(CT -> (none); MfrId Toshiba -> (none)
Changed lines of the file:
@@
 F 2 "Capacitors_SMD:C_0805" H 7888 4550 30  0001 C CNN
 F 3 "http://www.murata.com/~/media/webrenewal/support/library/catalog/products/capacitor/mlcc/c02e.ashx" H 7850 4700 60  0001 C CNN
-F 4 "GRM219R61H105KA73D" H 7900 4500 39  0001 L BNN "MfgId"
-F 5 "Murata" H 7850 4700 60  0001 C CNN "MfrId"
+F 4 "GRM219R61H105KA73D" H 7900 4500 39  0001 L BNN "Mfg1Id"
+F 5 "Murata" H 7850 4700 60  0001 C CNN "Mfg1"
 F 6 "Digikey" H 7850 4700 60  0001 C CNN "Vend1"
 F 7 "490-10743-2-ND" H 7850 4700 60  0001 C CNN "Vend1Id"
@@
 F 5 "490-9672-2-ND" V 6150 4600 60  0001 C CNN "Vend1Id"
 F 6 "Digikey" V 6150 4600 60  0001 C CNN "Vend1"
-F 7 "Murata" V 6150 4600 60  0001 C CNN "MfrId"
-F 8 "GRM21BR71H104MA01L" V 6150 4600 60  0001 C CNN "MfgId"
+F 7 "Murata" V 6150 4600 60  0001 C CNN "Mfg1"
+F 8 "GRM21BR71H104MA01L" V 6150 4600 60  0001 C CNN "Mfg1Id"
 	1    6150 4600
 	-1   0    0    1
@@
 F 4 "TCR2EF12LM(CTCT-ND" H 7100 4400 60  0001 C CNN "Vend1Id"
 F 5 "Digikey" H 7100 4400 60  0001 C CNN "Vend1"
-F 6 "Toshiba" H 7100 4400 60  0001 C CNN "MfrId"
-F 7 "TCR2EF12.LM(CT" H 7100 4400 60  0001 C CNN "MfgId"
+F 6 "Toshiba" H 7100 4400 60  0001 C CNN "Mfg1"
+F 7 "TCR2EF12.LM(CT" H 7100 4400 60  0001 C CNN "Mfg1Id"
 F 8 "LDO 1.2V 200mA" H 7000 3850 39  0000 C CNN "Description"
 F 9 "0.07110" H 7100 4400 60  0001 C CNN "RefPrice1k"
@@
 F 2 "Capacitors_SMD:C_0805" H 5188 4550 30  0001 C CNN
 F 3 "http://www.murata.com/~/media/webrenewal/support/library/catalog/products/capacitor/mlcc/c02e.ashx" H 5150 4700 60  0001 C CNN
-F 4 "GRM219R61H105KA73D" H 5200 4500 39  0001 L BNN "MfgId"
-F 5 "Murata" H 5150 4700 60  0001 C CNN "MfrId"
+F 4 "GRM219R61H105KA73D" H 5200 4500 39  0001 L BNN "Mfg1Id"
+F 5 "Murata" H 5150 4700 60  0001 C CNN "Mfg1"
 F 6 "Digikey" H 5150 4700 60  0001 C CNN "Vend1"
 F 7 "490-10743-2-ND" H 5150 4700 60  0001 C CNN "Vend1Id"
@@
 F 5 "490-9672-2-ND" V 3450 4600 60  0001 C CNN "Vend1Id"
 F 6 "Digikey" V 3450 4600 60  0001 C CNN "Vend1"
-F 7 "Murata" V 3450 4600 60  0001 C CNN "MfrId"
-F 8 "GRM21BR71H104MA01L" V 3450 4600 60  0001 C CNN "MfgId"
+F 7 "Murata" V 3450 4600 60  0001 C CNN "Mfg1"
+F 8 "GRM21BR71H104MA01L" V 3450 4600 60  0001 C CNN "Mfg1Id"
 	1    3450 4600
 	-1   0    0    1
@@
 F 4 "TCR2EF25LM(CTCT-ND" H 4400 4400 60  0001 C CNN "Vend1Id"
 F 5 "Digikey" H 4400 4400 60  0001 C CNN "Vend1"
-F 6 "Toshiba" H 4400 4400 60  0001 C CNN "MfrId"
-F 7 "TCR2EF25.LM(CT" H 4400 4400 60  0001 C CNN "MfgId"
+F 6 "Toshiba" H 4400 4400 60  0001 C CNN "Mfg1"
+F 7 "TCR2EF25.LM(CT" H 4400 4400 60  0001 C CNN "Mfg1Id"
 F 8 "LDO 2.5V 200mA" H 4300 3850 39  0000 C CNN "Description"
 F 9 "0.07110" H 4400 4400 60  0001 C CNN "RefPrice1k"
@@
 72 0F 1C A9 DC 70 49 CB 79 33 88 85 99 AD 01 6C 4B 10 FC 3B 13 DE 3B 37 68 79 AD 07 BC 00 3C 0E
 3C 31 EE E3 D8 E7 0F 03 D7 7B 9F FB C1 E1 FF 01 18 C4 96 1D B8 0E 40 07 00 00 00 00 49 45 4E 44
-AE 42 60 82 44
+AE 42 60 82 B0
 EndData
 $EndBitmap
