File: boards/spine/power-ldo.sch (KiCad schematic (older format))
At the start: 6 parts, among them U13 TCR2EF25, U14 TCR2EF12

Commit message: Capacitor upgrades, BOM tidying
Parts:
- renumbered C74 to C75, C75 to C76, C76 to C77, C77 to C78, U13 to U12, U14 to U13
Changed lines of the file:
@@
 $EndDescr
 $Comp
-L C C77
+L C C78
 U 1 1 564D1EB4
 P 7850 4700
-F 0 "C77" H 7900 4800 50  0000 L CNN
+F 0 "C78" H 7900 4800 50  0000 L CNN
 F 1 "1uF " H 7900 4600 50  0000 L CNN
 F 2 "Capacitors_SMD:C_0805" H 7888 4550 30  0001 C CNN
@@
 $EndComp
 $Comp
-L C C76
+L C C77
 U 1 1 564D1EB5
 P 6150 4600
-F 0 "C76" H 6000 4500 50  0000 L CNN
+F 0 "C77" H 6000 4500 50  0000 L CNN
 F 1 "0.1uF" H 5900 4700 50  0000 L CNN
 F 2 "Capacitors_SMD:C_0805" H 6188 4450 30  0001 C CNN
@@
 $EndComp
 $Comp
-L TCR2EF U14
+L TCR2EF U13
 U 1 1 564D1EB8
 P 7100 4400
-F 0 "U14" H 6750 4550 60  0000 L CNN
+F 0 "U13" H 6750 4550 60  0000 L CNN
 F 1 "TCR2EF12" H 6750 3950 60  0000 L CNN
 F 2 "TO_SOT_Packages_SMD:SOT-23-5" H 7000 4550 60  0001 C CNN
@@
 $EndComp
 $Comp
-L GND #PWR0143
+L GND #PWR159
 U 1 1 564D1EB9
 P 7850 4950
-F 0 "#PWR0143" H 7850 4700 50  0001 C CNN
+F 0 "#PWR159" H 7850 4700 50  0001 C CNN
 F 1 "GND" H 7850 4800 50  0000 C CNN
 F 2 "" H 7850 4950 60  0000 C CNN
@@
 NoConn ~ 7650 4550
 $Comp
-L GND #PWR0144
+L GND #PWR157
 U 1 1 564D1EBA
 P 6150 5000
-F 0 "#PWR0144" H 6150 4750 50  0001 C CNN
+F 0 "#PWR157" H 6150 4750 50  0001 C CNN
 F 1 "GND" H 6150 4850 50  0000 C CNN
 F 2 "" H 6150 5000 60  0000 C CNN
@@
 $EndComp
 $Comp
-L C C75
+L C C76
 U 1 1 564D1EBB
 P 5150 4700
-F 0 "C75" H 5200 4800 50  0000 L CNN
+F 0 "C76" H 5200 4800 50  0000 L CNN
 F 1 "1uF " H 5200 4600 50  0000 L CNN
 F 2 "Capacitors_SMD:C_0805" H 5188 4550 30  0001 C CNN
@@
 $EndComp
 $Comp
-L C C74
+L C C75
 U 1 1 564D1EBC
 P 3450 4600
-F 0 "C74" H 3300 4500 50  0000 L CNN
+F 0 "C75" H 3300 4500 50  0000 L CNN
 F 1 "0.1uF" H 3200 4700 50  0000 L CNN
 F 2 "Capacitors_SMD:C_0805" H 3488 4450 30  0001 C CNN
@@
 $EndComp
 $Comp
-L TCR2EF U13
+L TCR2EF U12
 U 1 1 564D1EBD
 P 4400 4400
-F 0 "U13" H 4050 4550 60  0000 L CNN
+F 0 "U12" H 4050 4550 60  0000 L CNN
 F 1 "TCR2EF25" H 4050 3950 60  0000 L CNN
 F 2 "TO_SOT_Packages_SMD:SOT-23-5" H 4300 4550 60  0001 C CNN
@@
 $EndComp
 $Comp
-L GND #PWR0145
+L GND #PWR156
 U 1 1 564D1EBE
 P 5150 4950
-F 0 "#PWR0145" H 5150 4700 50  0001 C CNN
+F 0 "#PWR156" H 5150 4700 50  0001 C CNN
 F 1 "GND" H 5150 4800 50  0000 C CNN
 F 2 "" H 5150 4950 60  0000 C CNN
@@
 NoConn ~ 4950 4550
 $Comp
-L GND #PWR0146
+L GND #PWR154
 U 1 1 564D1EBF
 P 3450 5000
-F 0 "#PWR0146" H 3450 4750 50  0001 C CNN
+F 0 "#PWR154" H 3450 4750 50  0001 C CNN
 F 1 "GND" H 3450 4850 50  0000 C CNN
 F 2 "" H 3450 5000 60  0000 C CNN
@@
 $EndComp
 $Comp
-L +2V5 #PWR0147
+L +2V5 #PWR155
 U 1 1 564D1EC0
 P 5150 4300
-F 0 "#PWR0147" H 5150 4150 50  0001 C CNN
+F 0 "#PWR155" H 5150 4150 50  0001 C CNN
 F 1 "+2V5" H 5150 4440 50  0000 C CNN
 F 2 "" H 5150 4300 60  0000 C CNN
@@
 2.5v = FPGA NVCM programming voltage\n\n(Some circuits approximate this with a diode\ndrop from 3.3v, but that's pretty dirty and\nthese LDOs are about as cheap as a diode.)
 $Comp
-L +3.3V #PWR0148
+L +3.3V #PWR153
 U 1 1 564D1EC2
 P 3450 4300
-F 0 "#PWR0148" H 3450 4150 50  0001 C CNN
+F 0 "#PWR153" H 3450 4150 50  0001 C CNN
 F 1 "+3.3V" H 3450 4440 50  0000 C CNN
 F 2 "" H 3450 4300 60  0000 C CNN
@@
 $EndComp
 $Comp
-L +1V2 #PWR0149
+L +1V2 #PWR158
 U 1 1 564D1EC3
 P 7850 4300
-F 0 "#PWR0149" H 7850 4150 50  0001 C CNN
+F 0 "#PWR158" H 7850 4150 50  0001 C CNN
 F 1 "+1V2" H 7850 4440 50  0000 C CNN
 F 2 "" H 7850 4300 60  0000 C CNN
@@
 FB 59 00 E6 A5 69 3A 37 9E CF 73 BC F7 37 E3 33 5D 9E A8 3E 7F 80 FA F7 F6 BB 44 F4 6E D4 E7 77
 A2 1E 1F 27 A2 E3 16 70 32 E9 54 FE 3F E7 AF 00 CA 1C A3 36 0A 00 00 00 00 49 45 4E 44 AE 42 60
-82 00
+82 7E
 EndData
 $EndBitmap
@@
 72 0F 1C A9 DC 70 49 CB 79 33 88 85 99 AD 01 6C 4B 10 FC 3B 13 DE 3B 37 68 79 AD 07 BC 00 3C 0E
 3C 31 EE E3 D8 E7 0F 03 D7 7B 9F FB C1 E1 FF 01 18 C4 96 1D B8 0E 40 07 00 00 00 00 49 45 4E 44
-AE 42 60 82 B0
+AE 42 60 82 10
 EndData
 $EndBitmap

Commit message: Schematics stabilizing for next proto, starting PCB updates
Parts:
- renumbered C75 to C74, C76 to C75, C77 to C76, C78 to C77
Changed lines of the file:
@@
 $EndDescr
 $Comp
-L C C78
+L C C77
 U 1 1 564D1EB4
 P 7850 4700
-F 0 "C78" H 7900 4800 50  0000 L CNN
+F 0 "C77" H 7900 4800 50  0000 L CNN
 F 1 "1uF " H 7900 4600 50  0000 L CNN
 F 2 "Capacitors_SMD:C_0805" H 7888 4550 30  0001 C CNN
@@
 $EndComp
 $Comp
-L C C77
+L C C76
 U 1 1 564D1EB5
 P 6150 4600
-F 0 "C77" H 6000 4500 50  0000 L CNN
+F 0 "C76" H 6000 4500 50  0000 L CNN
 F 1 "0.1uF" H 5900 4700 50  0000 L CNN
 F 2 "Capacitors_SMD:C_0805" H 6188 4450 30  0001 C CNN
@@
 $EndComp
 $Comp
-L C C76
+L C C75
 U 1 1 564D1EBB
 P 5150 4700
-F 0 "C76" H 5200 4800 50  0000 L CNN
+F 0 "C75" H 5200 4800 50  0000 L CNN
 F 1 "1uF " H 5200 4600 50  0000 L CNN
 F 2 "Capacitors_SMD:C_0805" H 5188 4550 30  0001 C CNN
@@
 $EndComp
 $Comp
-L C C75
+L C C74
 U 1 1 564D1EBC
 P 3450 4600
-F 0 "C75" H 3300 4500 50  0000 L CNN
+F 0 "C74" H 3300 4500 50  0000 L CNN
 F 1 "0.1uF" H 3200 4700 50  0000 L CNN
 F 2 "Capacitors_SMD:C_0805" H 3488 4450 30  0001 C CNN
@@
 FB 59 00 E6 A5 69 3A 37 9E CF 73 BC F7 37 E3 33 5D 9E A8 3E 7F 80 FA F7 F6 BB 44 F4 6E D4 E7 77
 A2 1E 1F 27 A2 E3 16 70 32 E9 54 FE 3F E7 AF 00 CA 1C A3 36 0A 00 00 00 00 49 45 4E 44 AE 42 60
-82 00
+82 70
 EndData
 $EndBitmap
@@
 72 0F 1C A9 DC 70 49 CB 79 33 88 85 99 AD 01 6C 4B 10 FC 3B 13 DE 3B 37 68 79 AD 07 BC 00 3C 0E
 3C 31 EE E3 D8 E7 0F 03 D7 7B 9F FB C1 E1 FF 01 18 C4 96 1D B8 0E 40 07 00 00 00 00 49 45 4E 44
-AE 42 60 82 01
+AE 42 60 82 00
 EndData
 $EndBitmap
