File: boards/spine/spine-clock.sch (KiCad schematic (older format))
At the start: 8 parts, among them U15 Si5351B, X1 25.0000 MHz 15ppm 8pF

Commit message: BOM cleanup
Especially fix the confusing and mostly incorrect Mfg/Mfr stuff that I inherited from somewhere.
Parts:
- C78, C79: Mfg1 (none) -> Murata; Mfg1Id (none) -> GRM21BR71H104MA01L; MfgId GRM21BR71H104MA01L -> (none); MfrId Murata -> (none)
- C80: Mfg1 (none) -> Murata; Mfg1Id (none) -> GRM219R61H105KA73D; MfgId GRM219R61H105KA73D -> (none); MfrId Murata -> (none)
- R34, R35: Mfg1 (none) -> Stackpole; Mfg1Id (none) -> RMCF0805JT2K20CT; MfgId RMCF0805JT2K20CT -> (none); MfrId Stackpole -> (none)
- R36: Mfg1 (none) -> Stackpole; Mfg1Id (none) -> RMCF0805JT10K0; MfgId RMCF0805JT10K0 -> (none); MfrId Stackpole -> (none)
- U15: Mfg1 (none) -> Silicon Labs; Mfg1Id (none) -> SI5351B-B-GM; MfgId Silicon Labs -> (none); MfrId SI5351B-B-GM -> (none)
- X1: Mfg1 (none) -> NDK; Mfg1Id (none) -> NX3225SA-25.000M-STD-CSR-3; MfgId NDK -> (none); MfrId NX3225SA-25.000M-STD-CSR-3 -> (none)
Changed lines of the file:
@@
 F 4 "Digikey" H 5850 3250 60  0001 C CNN "Vend1"
 F 5 "336-2401-5-ND" H 5850 3250 60  0001 C CNN "Vend1Id"
-F 6 "Silicon Labs" H 5850 3250 60  0001 C CNN "MfgId"
-F 7 "SI5351B-B-GM" H 5850 3250 60  0001 C CNN "MfrId"
+F 6 "Silicon Labs" H 5850 3250 60  0001 C CNN "Mfg1"
+F 7 "SI5351B-B-GM" H 5850 3250 60  0001 C CNN "Mfg1Id"
 F 8 "2.01798" H 5850 3250 60  0001 C CNN "RefPrice1k"
 	1    5850 3250
@@
 F 5 "RMCF0805JT2K20CT-ND" V 4150 3600 60  0001 C CNN "Vend1Id"
 F 6 "Digikey" V 4150 3600 60  0001 C CNN "Vend1"
-F 7 "Stackpole" V 4150 3600 60  0001 C CNN "MfrId"
-F 8 "RMCF0805JT2K20CT" V 4150 3600 60  0001 C CNN "MfgId"
+F 7 "Stackpole" V 4150 3600 60  0001 C CNN "Mfg1"
+F 8 "RMCF0805JT2K20CT" V 4150 3600 60  0001 C CNN "Mfg1Id"
 	1    4150 3600
 	1    0    0    -1
@@
 F 4 "Digikey" H 4900 3400 60  0001 C CNN "Vend1"
 F 5 "644-1267-1-ND" H 4900 3400 60  0001 C CNN "Vend1Id"
-F 6 "NDK" H 4900 3400 60  0001 C CNN "MfgId"
-F 7 "NX3225SA-25.000M-STD-CSR-3" H 4900 3400 60  0001 C CNN "MfrId"
+F 6 "NDK" H 4900 3400 60  0001 C CNN "Mfg1"
+F 7 "NX3225SA-25.000M-STD-CSR-3" H 4900 3400 60  0001 C CNN "Mfg1Id"
 F 8 "0.4187" H 4900 3400 60  0001 C CNN "RefPrice1k"
 	1    4900 3400
@@
 F 5 "RMCF0805JT2K20CT-ND" V 3950 3600 60  0001 C CNN "Vend1Id"
 F 6 "Digikey" V 3950 3600 60  0001 C CNN "Vend1"
-F 7 "Stackpole" V 3950 3600 60  0001 C CNN "MfrId"
-F 8 "RMCF0805JT2K20CT" V 3950 3600 60  0001 C CNN "MfgId"
+F 7 "Stackpole" V 3950 3600 60  0001 C CNN "Mfg1"
+F 8 "RMCF0805JT2K20CT" V 3950 3600 60  0001 C CNN "Mfg1Id"
 	1    3950 3600
 	1    0    0    -1
@@
 F 5 "RMCF0805JT10K0CT-ND" V 4450 3850 60  0001 C CNN "Vend1Id"
 F 6 "Digikey" V 4450 3850 60  0001 C CNN "Vend1"
-F 7 "Stackpole" V 4450 3850 60  0001 C CNN "MfrId"
-F 8 "RMCF0805JT10K0" V 4450 3850 60  0001 C CNN "MfgId"
+F 7 "Stackpole" V 4450 3850 60  0001 C CNN "Mfg1"
+F 8 "RMCF0805JT10K0" V 4450 3850 60  0001 C CNN "Mfg1Id"
 	1    4450 3850
 	0    -1   -1   0
@@
 F 5 "490-9672-2-ND" V 3650 5350 60  0001 C CNN "Vend1Id"
 F 6 "Digikey" V 3650 5350 60  0001 C CNN "Vend1"
-F 7 "Murata" V 3650 5350 60  0001 C CNN "MfrId"
-F 8 "GRM21BR71H104MA01L" V 3650 5350 60  0001 C CNN "MfgId"
+F 7 "Murata" V 3650 5350 60  0001 C CNN "Mfg1"
+F 8 "GRM21BR71H104MA01L" V 3650 5350 60  0001 C CNN "Mfg1Id"
 	1    3650 5350
 	-1   0    0    1
@@
 F 2 "Capacitors_SMD:C_0805" H 4788 4250 30  0001 C CNN
 F 3 "http://www.murata.com/~/media/webrenewal/support/library/catalog/products/capacitor/mlcc/c02e.ashx" H 4750 4400 60  0001 C CNN
-F 4 "GRM219R61H105KA73D" H 4800 4200 39  0001 L BNN "MfgId"
-F 5 "Murata" H 4750 4400 60  0001 C CNN "MfrId"
+F 4 "GRM219R61H105KA73D" H 4800 4200 39  0001 L BNN "Mfg1Id"
+F 5 "Murata" H 4750 4400 60  0001 C CNN "Mfg1"
 F 6 "Digikey" H 4750 4400 60  0001 C CNN "Vend1"
 F 7 "490-10743-2-ND" H 4750 4400 60  0001 C CNN "Vend1Id"
@@
 F 5 "490-9672-2-ND" V 4050 5350 60  0001 C CNN "Vend1Id"
 F 6 "Digikey" V 4050 5350 60  0001 C CNN "Vend1"
-F 7 "Murata" V 4050 5350 60  0001 C CNN "MfrId"
-F 8 "GRM21BR71H104MA01L" V 4050 5350 60  0001 C CNN "MfgId"
+F 7 "Murata" V 4050 5350 60  0001 C CNN "Mfg1"
+F 8 "GRM21BR71H104MA01L" V 4050 5350 60  0001 C CNN "Mfg1Id"
 	1    4050 5350
 	-1   0    0    1
@@
 72 0F 1C A9 DC 70 49 CB 79 33 88 85 99 AD 01 6C 4B 10 FC 3B 13 DE 3B 37 68 79 AD 07 BC 00 3C 0E
 3C 31 EE E3 D8 E7 0F 03 D7 7B 9F FB C1 E1 FF 01 18 C4 96 1D B8 0E 40 07 00 00 00 00 49 45 4E 44
-AE 42 60 82 FF
+AE 42 60 82 00
 EndData
 $EndBitmap

Commit message: Capacitor upgrades, BOM tidying
Parts:
- renumbered C78 to C79, C79 to C80, C80 to C81, R34 to R36, R35 to R37, R36 to R38, U15 to U14, X1 to X2
Changed lines of the file:
@@
 CLK[7..0]
 $Comp
-L Si5351B U15
+L Si5351B U14
 U 1 1 564F7EE6
 P 5850 3250
-F 0 "U15" H 5600 3000 60  0000 L CNN
+F 0 "U14" H 5600 3000 60  0000 L CNN
 F 1 "Si5351B" H 5600 2900 60  0000 L CNN
 F 2 "Housings_DFN_QFN:QFN-20-1EP_4x4mm_Pitch0.5mm" H 5850 3250 60  0001 C CNN
@@
 $EndComp
 $Comp
-L GND #PWR0150
+L GND #PWR167
 U 1 1 564F7F28
 P 5650 4550
-F 0 "#PWR0150" H 5650 4300 50  0001 C CNN
+F 0 "#PWR167" H 5650 4300 50  0001 C CNN
 F 1 "GND" H 5650 4400 50  0000 C CNN
 F 2 "" H 5650 4550 60  0000 C CNN
@@
 $EndComp
 $Comp
-L +3.3V #PWR0151
+L +3.3V #PWR166
 U 1 1 564F7F3F
 P 5550 2600
-F 0 "#PWR0151" H 5550 2450 50  0001 C CNN
+F 0 "#PWR166" H 5550 2450 50  0001 C CNN
 F 1 "+3.3V" H 5550 2740 50  0000 C CNN
 F 2 "" H 5550 2600 60  0000 C CNN
@@
 CLK7
 $Comp
-L R R35
+L R R37
 U 1 1 564F965E
 P 4150 3600
-F 0 "R35" V 4230 3600 50  0000 C CNN
+F 0 "R37" V 4230 3600 50  0000 C CNN
 F 1 "2.2k" V 4150 3600 50  0000 C CNN
 F 2 "Resistors_SMD:R_0805" V 4080 3600 30  0001 C CNN
@@
 $EndComp
 $Comp
-L XTAL_CHIP32X25 X1
+L XTAL_CHIP32X25 X2
 U 1 1 564FA165
 P 4900 3400
-F 0 "X1" V 4900 3150 50  0000 R CNN
+F 0 "X2" V 4900 3150 50  0000 R CNN
 F 1 "25.0000 MHz 15ppm 8pF" V 4500 3300 39  0000 C CNN
 F 2 "Crystals:crystal_FA238-TSX3225" H 4900 3550 50  0001 C CNN
@@
 	4900 3650 5050 3650
 $Comp
-L GND #PWR0152
+L GND #PWR163
 U 1 1 564FA8B8
 P 4600 3300
-F 0 "#PWR0152" H 4600 3050 50  0001 C CNN
+F 0 "#PWR163" H 4600 3050 50  0001 C CNN
 F 1 "GND" V 4600 3100 50  0000 C CNN
 F 2 "" H 4600 3300 60  0000 C CNN
@@
 $EndComp
 $Comp
-L GND #PWR0153
+L GND #PWR168
 U 1 1 564FA968
 P 6650 4250
-F 0 "#PWR0153" H 6650 4000 50  0001 C CNN
+F 0 "#PWR168" H 6650 4000 50  0001 C CNN
 F 1 "GND" H 6650 4100 50  0000 C CNN
 F 2 "" H 6650 4250 60  0000 C CNN
@@
 Connection ~ 6650 4150
 $Comp
-L R R34
+L R R36
 U 1 1 564FABBB
 P 3950 3600
-F 0 "R34" V 4030 3600 50  0000 C CNN
+F 0 "R36" V 4030 3600 50  0000 C CNN
 F 1 "2.2k" V 3950 3600 50  0000 C CNN
 F 2 "Resistors_SMD:R_0805" V 3880 3600 30  0001 C CNN
@@
 $EndComp
 $Comp
-L +3.3V #PWR0154
+L +3.3V #PWR162
 U 1 1 564FABDD
 P 3950 3300
-F 0 "#PWR0154" H 3950 3150 50  0001 C CNN
+F 0 "#PWR162" H 3950 3150 50  0001 C CNN
 F 1 "+3.3V" H 3950 3440 50  0000 C CNN
 F 2 "" H 3950 3300 60  0000 C CNN
@@
 Connection ~ 3950 4050
 $Comp
-L R R36
+L R R38
 U 1 1 564FC56E
 P 4450 3850
-F 0 "R36" V 4530 3850 50  0000 C CNN
+F 0 "R38" V 4530 3850 50  0000 C CNN
 F 1 "10k" V 4450 3850 50  0000 C CNN
 F 2 "Resistors_SMD:R_0805" V 4380 3850 30  0001 C CNN
@@
 $EndComp
 $Comp
-L C C78
+L C C79
 U 1 1 564FC57D
 P 3650 5350
-F 0 "C78" H 3650 5250 50  0000 L CNN
+F 0 "C79" H 3650 5250 50  0000 L CNN
 F 1 "0.1uF" H 3650 5200 50  0000 L TNN
 F 2 "Capacitors_SMD:C_0805" H 3688 5200 30  0001 C CNN
@@
 $EndComp
 $Comp
-L C C80
+L C C81
 U 1 1 564FD614
 P 4750 4400
-F 0 "C80" H 4800 4500 50  0000 L CNN
+F 0 "C81" H 4800 4500 50  0000 L CNN
 F 1 "1uF " H 4800 4300 50  0000 L CNN
 F 2 "Capacitors_SMD:C_0805" H 4788 4250 30  0001 C CNN
@@
 $EndComp
 $Comp
-L GND #PWR0155
+L GND #PWR164
 U 1 1 564FE031
 P 4600 3500
-F 0 "#PWR0155" H 4600 3250 50  0001 C CNN
+F 0 "#PWR164" H 4600 3250 50  0001 C CNN
 F 1 "GND" H 4600 3350 50  0001 C CNN
 F 2 "" H 4600 3500 60  0000 C CNN
@@
 $EndComp
 $Comp
-L GND #PWR0156
+L GND #PWR165
 U 1 1 564FE16F
 P 4750 4550
-F 0 "#PWR0156" H 4750 4300 50  0001 C CNN
+F 0 "#PWR165" H 4750 4300 50  0001 C CNN
 F 1 "GND" H 4750 4400 50  0000 C CNN
 F 2 "" H 4750 4550 60  0000 C CNN
@@
 	4300 3850 3750 3850
 $Comp
-L +3.3V #PWR0157
+L +3.3V #PWR160
 U 1 1 564FE49E
 P 3650 5000
-F 0 "#PWR0157" H 3650 4850 50  0001 C CNN
+F 0 "#PWR160" H 3650 4850 50  0001 C CNN
 F 1 "+3.3V" H 3650 5140 50  0000 C CNN
 F 2 "" H 3650 5000 60  0000 C CNN
@@
 $EndComp
 $Comp
-L GND #PWR0158
+L GND #PWR161
 U 1 1 564FE4DC
 P 3650 5700
-F 0 "#PWR0158" H 3650 5450 50  0001 C CNN
+F 0 "#PWR161" H 3650 5450 50  0001 C CNN
 F 1 "GND" H 3650 5550 50  0000 C CNN
 F 2 "" H 3650 5700 60  0000 C CNN
@@
 	3650 5500 3650 5700
 $Comp
-L C C79
+L C C80
 U 1 1 564FE623
 P 4050 5350
-F 0 "C79" H 4050 5250 50  0000 L CNN
+F 0 "C80" H 4050 5250 50  0000 L CNN
 F 1 "0.1uF" H 4050 5200 50  0000 L TNN
 F 2 "Capacitors_SMD:C_0805" H 4088 5200 30  0001 C CNN

Commit message: Schematics stabilizing for next proto, starting PCB updates
Parts:
- renumbered C79 to C78, C80 to C79, C81 to C80
Changed lines of the file:
@@
 $EndComp
 $Comp
-L C C79
+L C C78
 U 1 1 564FC57D
 P 3650 5350
-F 0 "C79" H 3650 5250 50  0000 L CNN
+F 0 "C78" H 3650 5250 50  0000 L CNN
 F 1 "0.1uF" H 3650 5200 50  0000 L TNN
 F 2 "Capacitors_SMD:C_0805" H 3688 5200 30  0001 C CNN
@@
 $EndComp
 $Comp
-L C C81
+L C C80
 U 1 1 564FD614
 P 4750 4400
-F 0 "C81" H 4800 4500 50  0000 L CNN
+F 0 "C80" H 4800 4500 50  0000 L CNN
 F 1 "1uF " H 4800 4300 50  0000 L CNN
 F 2 "Capacitors_SMD:C_0805" H 4788 4250 30  0001 C CNN
@@
 	3650 5500 3650 5700
 $Comp
-L C C80
+L C C79
 U 1 1 564FE623
 P 4050 5350
-F 0 "C80" H 4050 5250 50  0000 L CNN
+F 0 "C79" H 4050 5250 50  0000 L CNN
 F 1 "0.1uF" H 4050 5200 50  0000 L TNN
 F 2 "Capacitors_SMD:C_0805" H 4088 5200 30  0001 C CNN
