File: boards/spine/power-usb-in.sch (KiCad schematic (older format))
At the start: 13 parts, among them Q3 IRFML8244, U11 SiP32408, U12 SiP32408

Commit message: More simplification and BOM optimization
Thanks for the hints on the ST485 and dual-FETs, @mikelectricstuf!
Parts:
- Q3: value IRFML8244 -> 2N7002P; MfgId IRFML8244TRPBF -> 2N7002P.215; MfrId Infineon -> NXP; RefPrice1k 0.1046 -> 0.02936; Vend1Id IRFML8244TRPBFCT-ND -> 568-5818-1-ND
Changed lines of the file:
@@
 U 1 1 564D4E76
 P 3600 4000
-F 0 "Q3" H 3900 4050 50  0000 R CNN
-F 1 "IRFML8244" H 4200 3950 50  0001 R CNN
+F 0 "Q3" H 3300 4100 50  0000 L CNN
+F 1 "2N7002P" H 3300 4200 50  0000 L CNN
 F 2 "TO_SOT_Packages_SMD:SOT-23" H 3800 4100 29  0001 C CNN
-F 3 "http://www.irf.com/product-info/datasheets/data/irfml8244pbf.pdf" H 3600 4000 60  0001 C CNN
-F 4 "Infineon" H 3600 4000 60  0001 C CNN "MfrId"
-F 5 "IRFML8244TRPBF" H 3600 4000 60  0001 C CNN "MfgId"
-F 6 "0.1046" H 3600 4000 60  0001 C CNN "RefPrice1k"
+F 3 "http://www.nxp.com/documents/data_sheet/2N7002P.pdf" H 3600 4000 60  0001 C CNN
+F 4 "NXP" H 3600 4000 60  0001 C CNN "MfrId"
+F 5 "2N7002P.215" H 3600 4000 60  0001 C CNN "MfgId"
+F 6 "0.02936" H 3600 4000 60  0001 C CNN "RefPrice1k"
 F 7 "Digikey" H 3600 4000 60  0001 C CNN "Vend1"
-F 8 "IRFML8244TRPBFCT-ND" H 3600 4000 60  0001 C CNN "Vend1Id"
+F 8 "568-5818-1-ND" H 3600 4000 60  0001 C CNN "Vend1Id"
 	1    3600 4000
 	1    0    0    -1
@@
 $EndComp
 $Comp
-L +5V #PWR137
+L +5V #PWR0135
 U 1 1 564D4EA6
 P 5900 2800
-F 0 "#PWR137" H 5900 2650 50  0001 C CNN
+F 0 "#PWR0135" H 5900 2650 50  0001 C CNN
 F 1 "+5V" H 5900 2940 50  0000 C CNN
 F 2 "" H 5900 2800 60  0000 C CNN
@@
 CONVERTED_5V_OKAY
 $Comp
-L GND #PWR135
+L GND #PWR0136
 U 1 1 564D0835
 P 3700 4550
-F 0 "#PWR135" H 3700 4300 50  0001 C CNN
+F 0 "#PWR0136" H 3700 4300 50  0001 C CNN
 F 1 "GND" H 3700 4400 50  0000 C CNN
 F 2 "" H 3700 4550 60  0000 C CNN
@@
 $EndComp
 $Comp
-L GND #PWR136
+L GND #PWR0137
 U 1 1 564D1BDA
 P 4600 6150
-F 0 "#PWR136" H 4600 5900 50  0001 C CNN
+F 0 "#PWR0137" H 4600 5900 50  0001 C CNN
 F 1 "GND" H 4600 6000 50  0000 C CNN
 F 2 "" H 4600 6150 60  0000 C CNN
@@
 $EndComp
 $Comp
-L GND #PWR138
+L GND #PWR0138
 U 1 1 564EBB09
 P 6850 3750
-F 0 "#PWR138" H 6850 3500 50  0001 C CNN
+F 0 "#PWR0138" H 6850 3500 50  0001 C CNN
 F 1 "GND" H 6850 3600 50  0000 C CNN
 F 2 "" H 6850 3750 60  0000 C CNN
@@
 FB 59 00 E6 A5 69 3A 37 9E CF 73 BC F7 37 E3 33 5D 9E A8 3E 7F 80 FA F7 F6 BB 44 F4 6E D4 E7 77
 A2 1E 1F 27 A2 E3 16 70 32 E9 54 FE 3F E7 AF 00 CA 1C A3 36 0A 00 00 00 00 49 45 4E 44 AE 42 60
-82 70
+82 00
 EndData
 $EndBitmap

Commit message: BOM cleanup
Especially fix the confusing and mostly incorrect Mfg/Mfr stuff that I inherited from somewhere.
Parts:
- C65, C68, C69: Mfg1 (none) -> Murata; Mfg1Id (none) -> GRM21BR71H104MA01L; MfgId GRM21BR71H104MA01L -> (none); MfrId Murata -> (none)
- C66, C67: Mfg1 (none) -> Murata; Mfg1Id (none) -> GRM219R61H105KA73D; MfgId GRM219R61H105KA73D -> (none); MfrId Murata -> (none)
- C70, C71: Mfg1 (none) -> Murata; Mfg1Id (none) -> GRM31CR61H106MA12L; MfgId GRM31CR61H106MA12L -> (none); MfrId Murata -> (none)
- D7: Mfg1 (none) -> ON Semi; Mfg1Id (none) -> MMBZ12VALT1G; MfgId MMBZ12VALT1G -> (none); MfrId ON Semi -> (none)
- Q3: Mfg1 (none) -> NXP; Mfg1Id (none) -> 2N7002P.215; MfgId 2N7002P.215 -> (none); MfrId NXP -> (none)
- R31: Mfg1 (none) -> Stackpole; Mfg1Id (none) -> RMCF0805JT100K; MfgId RMCF0805JT100K -> (none); MfrId Stackpole -> (none)
- R32: Mfg1 (none) -> Stackpole; Mfg1Id (none) -> RMCF0805JT2K20CT; MfgId RMCF0805JT2K20CT -> (none); MfrId Stackpole -> (none)
- U11, U12: Mfg1 (none) -> Vishay; Mfg1Id (none) -> SIP32408DNP-T1-GE4; MfgId Vishay -> (none); MfrId SIP32408DNP-T1-GE4 -> (none)

Commit message: Capacitor upgrades, BOM tidying
Parts:
- renumbered C65 to C66, C66 to C67, C67 to C68, C68 to C69, C69 to C70, C70 to C71, C71 to C72, D7 to D8, Q3 to Q2, R31 to R33, R32 to R34, U11 to U10, U12 to U11
Changed lines of the file:
@@
 $EndDescr
 $Comp
-L Q_NMOS_GSD Q3
+L Q_NMOS_GSD Q2
 U 1 1 564D4E76
 P 3600 4000
-F 0 "Q3" H 3300 4100 50  0000 L CNN
+F 0 "Q2" H 3300 4100 50  0000 L CNN
 F 1 "2N7002P" H 3300 4200 50  0000 L CNN
 F 2 "TO_SOT_Packages_SMD:SOT-23" H 3800 4100 29  0001 C CNN
@@
 $EndComp
 $Comp
-L C C66
+L C C67
 U 1 1 564D4E85
 P 4600 3500
-F 0 "C66" H 4650 3600 50  0000 L CNN
+F 0 "C67" H 4650 3600 50  0000 L CNN
 F 1 "1uF " H 4650 3400 50  0000 L CNN
 F 2 "Capacitors_SMD:C_0805" H 4638 3350 30  0001 C CNN
@@
 $EndComp
 $Comp
-L R R31
+L R R33
 U 1 1 564D4E87
 P 3300 3200
-F 0 "R31" V 3380 3200 50  0000 C CNN
+F 0 "R33" V 3380 3200 50  0000 C CNN
 F 1 "100k" V 3300 3200 50  0000 C CNN
 F 2 "Resistors_SMD:R_0805" V 3230 3200 30  0001 C CNN
@@
 $EndComp
 $Comp
-L C C68
+L C C69
 U 1 1 564D4E88
 P 5900 3350
-F 0 "C68" H 5750 3250 50  0000 L CNN
+F 0 "C69" H 5750 3250 50  0000 L CNN
 F 1 "0.1uF" H 5650 3450 50  0000 L CNN
 F 2 "Capacitors_SMD:C_0805" H 5938 3200 30  0001 C CNN
@@
 $EndComp
 $Comp
-L +5V #PWR0135
+L +5V #PWR147
 U 1 1 564D4EA6
 P 5900 2800
-F 0 "#PWR0135" H 5900 2650 50  0001 C CNN
+F 0 "#PWR147" H 5900 2650 50  0001 C CNN
 F 1 "+5V" H 5900 2940 50  0000 C CNN
 F 2 "" H 5900 2800 60  0000 C CNN
@@
 CONVERTED_5V_OKAY
 $Comp
-L GND #PWR0136
+L GND #PWR145
 U 1 1 564D0835
 P 3700 4550
-F 0 "#PWR0136" H 3700 4300 50  0001 C CNN
+F 0 "#PWR145" H 3700 4300 50  0001 C CNN
 F 1 "GND" H 3700 4400 50  0000 C CNN
 F 2 "" H 3700 4550 60  0000 C CNN
@@
 When USB power is available, route it to the +5V rail\n(with reverse current protection)\n\nWhen/if external 5V becomes available, switch to it\nsoftly, then draw no power from upstream USB.
 $Comp
-L C C65
+L C C66
 U 1 1 564D0CD8
 P 4150 3500
-F 0 "C65" H 4000 3400 50  0000 L CNN
+F 0 "C66" H 4000 3400 50  0000 L CNN
 F 1 "0.1uF" H 3900 3600 50  0000 L CNN
 F 2 "Capacitors_SMD:C_0805" H 4188 3350 30  0001 C CNN
@@
 $EndComp
 $Comp
-L C C67
+L C C68
 U 1 1 564D1BB4
 P 4600 5700
-F 0 "C67" H 4650 5800 50  0000 L CNN
+F 0 "C68" H 4650 5800 50  0000 L CNN
 F 1 "1uF " H 4650 5600 50  0000 L CNN
 F 2 "Capacitors_SMD:C_0805" H 4638 5550 30  0001 C CNN
@@
 $EndComp
 $Comp
-L C C69
+L C C70
 U 1 1 564D1BBF
 P 5900 5550
-F 0 "C69" H 5750 5450 50  0000 L CNN
+F 0 "C70" H 5750 5450 50  0000 L CNN
 F 1 "0.1uF" H 5650 5650 50  0000 L CNN
 F 2 "Capacitors_SMD:C_0805" H 5938 5400 30  0001 C CNN
@@
 $EndComp
 $Comp
-L GND #PWR0137
+L GND #PWR146
 U 1 1 564D1BDA
 P 4600 6150
-F 0 "#PWR0137" H 4600 5900 50  0001 C CNN
+F 0 "#PWR146" H 4600 5900 50  0001 C CNN
 F 1 "GND" H 4600 6000 50  0000 C CNN
 F 2 "" H 4600 6150 60  0000 C CNN
@@
 $EndComp
 $Comp
-L R R32
+L R R34
 U 1 1 564D30A7
 P 3700 3500
-F 0 "R32" V 3780 3500 50  0000 C CNN
+F 0 "R34" V 3780 3500 50  0000 C CNN
 F 1 "2.2k" V 3700 3500 50  0000 C CNN
 F 2 "Resistors_SMD:R_0805" V 3630 3500 30  0001 C CNN
@@
 (High-Z logic input)
 $Comp
-L SiP32408 U11
+L SiP32408 U10
 U 1 1 564E43D8
 P 5150 2950
-F 0 "U11" H 4900 3250 60  0000 L CNN
+F 0 "U10" H 4900 3250 60  0000 L CNN
 F 1 "SiP32408" H 4900 3150 60  0000 L CNN
 F 2 "TDFN4:TDFN4" H 5200 3150 60  0001 C CNN
@@
 $EndComp
 $Comp
-L SiP32408 U12
+L SiP32408 U11
 U 1 1 564E481C
 P 5150 5150
-F 0 "U12" H 4900 5450 60  0000 L CNN
+F 0 "U11" H 4900 5450 60  0000 L CNN
 F 1 "SiP32408" H 4900 5350 60  0000 L CNN
 F 2 "TDFN4:TDFN4" H 5200 5350 60  0001 C CNN
@@
 $EndComp
 $Comp
-L C C70
+L C C71
 U 1 1 564EBB05
 P 6850 3200
-F 0 "C70" V 6800 3300 50  0000 L CNN
+F 0 "C71" V 6800 3300 50  0000 L CNN
 F 1 "10uF " V 6800 2900 50  0000 L CNN
 F 2 "Capacitors_SMD:C_1206" H 6888 3050 30  0001 C CNN
@@
 $EndComp
 $Comp
-L C C71
+L C C72
 U 1 1 564EBB06
 P 7100 3200
-F 0 "C71" V 7050 3300 50  0000 L CNN
+F 0 "C72" V 7050 3300 50  0000 L CNN
 F 1 "10uF " V 7050 2900 50  0000 L CNN
 F 2 "Capacitors_SMD:C_1206" H 7138 3050 30  0001 C CNN
@@
 $EndComp
 $Comp
-L GND #PWR0138
+L GND #PWR148
 U 1 1 564EBB09
 P 6850 3750
-F 0 "#PWR0138" H 6850 3500 50  0001 C CNN
+F 0 "#PWR148" H 6850 3500 50  0001 C CNN
 F 1 "GND" H 6850 3600 50  0000 C CNN
 F 2 "" H 6850 3750 60  0000 C CNN
@@
 FB 59 00 E6 A5 69 3A 37 9E CF 73 BC F7 37 E3 33 5D 9E A8 3E 7F 80 FA F7 F6 BB 44 F4 6E D4 E7 77
 A2 1E 1F 27 A2 E3 16 70 32 E9 54 FE 3F E7 AF 00 CA 1C A3 36 0A 00 00 00 00 49 45 4E 44 AE 42 60
-82 70
+82 00
 EndData
 $EndBitmap
@@
 72 0F 1C A9 DC 70 49 CB 79 33 88 85 99 AD 01 6C 4B 10 FC 3B 13 DE 3B 37 68 79 AD 07 BC 00 3C 0E
 3C 31 EE E3 D8 E7 0F 03 D7 7B 9F FB C1 E1 FF 01 18 C4 96 1D B8 0E 40 07 00 00 00 00 49 45 4E 44
-AE 42 60 82 B0
+AE 42 60 82 00
 EndData
 $EndBitmap
@@
 Transient clamping
 $Comp
-L D_Schottky_x2_ACom_KKA D7
+L D_Schottky_x2_ACom_KKA D8
 U 1 1 564EBB0D
 P 7800 3250
-F 0 "D7" H 8000 3450 50  0000 R CNN
+F 0 "D8" H 8000 3450 50  0000 R CNN
 F 1 "8.5VWM" H 7550 3450 50  0000 L CNN
 F 2 "TO_SOT_Packages_SMD:SOT-23" H 7800 3250 60  0001 C CNN

Commit message: Schematics stabilizing for next proto, starting PCB updates
Parts:
- renumbered C66 to C65, C67 to C66, C68 to C67, C69 to C68, C70 to C69, C71 to C70, C72 to C71
Changed lines of the file:
@@
 $EndComp
 $Comp
-L C C67
+L C C66
 U 1 1 564D4E85
 P 4600 3500
-F 0 "C67" H 4650 3600 50  0000 L CNN
+F 0 "C66" H 4650 3600 50  0000 L CNN
 F 1 "1uF " H 4650 3400 50  0000 L CNN
 F 2 "Capacitors_SMD:C_0805" H 4638 3350 30  0001 C CNN
@@
 $EndComp
 $Comp
-L C C69
+L C C68
 U 1 1 564D4E88
 P 5900 3350
-F 0 "C69" H 5750 3250 50  0000 L CNN
+F 0 "C68" H 5750 3250 50  0000 L CNN
 F 1 "0.1uF" H 5650 3450 50  0000 L CNN
 F 2 "Capacitors_SMD:C_0805" H 5938 3200 30  0001 C CNN
@@
 When USB power is available, route it to the +5V rail\n(with reverse current protection)\n\nWhen/if external 5V becomes available, switch to it\nsoftly, then draw no power from upstream USB.
 $Comp
-L C C66
+L C C65
 U 1 1 564D0CD8
 P 4150 3500
-F 0 "C66" H 4000 3400 50  0000 L CNN
+F 0 "C65" H 4000 3400 50  0000 L CNN
 F 1 "0.1uF" H 3900 3600 50  0000 L CNN
 F 2 "Capacitors_SMD:C_0805" H 4188 3350 30  0001 C CNN
@@
 $EndComp
 $Comp
-L C C68
+L C C67
 U 1 1 564D1BB4
 P 4600 5700
-F 0 "C68" H 4650 5800 50  0000 L CNN
+F 0 "C67" H 4650 5800 50  0000 L CNN
 F 1 "1uF " H 4650 5600 50  0000 L CNN
 F 2 "Capacitors_SMD:C_0805" H 4638 5550 30  0001 C CNN
@@
 $EndComp
 $Comp
-L C C70
+L C C69
 U 1 1 564D1BBF
 P 5900 5550
-F 0 "C70" H 5750 5450 50  0000 L CNN
+F 0 "C69" H 5750 5450 50  0000 L CNN
 F 1 "0.1uF" H 5650 5650 50  0000 L CNN
 F 2 "Capacitors_SMD:C_0805" H 5938 5400 30  0001 C CNN
@@
 $EndComp
 $Comp
-L C C71
+L C C70
 U 1 1 564EBB05
 P 6850 3200
-F 0 "C71" V 6800 3300 50  0000 L CNN
+F 0 "C70" V 6800 3300 50  0000 L CNN
 F 1 "10uF " V 6800 2900 50  0000 L CNN
 F 2 "Capacitors_SMD:C_1206" H 6888 3050 30  0001 C CNN
@@
 $EndComp
 $Comp
-L C C72
+L C C71
 U 1 1 564EBB06
 P 7100 3200
-F 0 "C72" V 7050 3300 50  0000 L CNN
+F 0 "C71" V 7050 3300 50  0000 L CNN
 F 1 "10uF " V 7050 2900 50  0000 L CNN
 F 2 "Capacitors_SMD:C_1206" H 7138 3050 30  0001 C CNN
@@
 72 0F 1C A9 DC 70 49 CB 79 33 88 85 99 AD 01 6C 4B 10 FC 3B 13 DE 3B 37 68 79 AD 07 BC 00 3C 0E
 3C 31 EE E3 D8 E7 0F 03 D7 7B 9F FB C1 E1 FF 01 18 C4 96 1D B8 0E 40 07 00 00 00 00 49 45 4E 44
-AE 42 60 82 A3
+AE 42 60 82 00
 EndData
 $EndBitmap
